Commit message: test base urdf fixes

File: mirte_base_control/bringup/urdf/base.urdf.xacro (robot description, xacro)
@@ -2,8 +2,8 @@
 <!-- Basic differential drive mobile base -->
 <robot xmlns:xacro="http://www.ros.org/wiki/xacro" name="diffdrive_robot">
-    <xacro:property name="yaml_param_file" value="$(find mirte_base_control)/config/control_master.yaml"/>
-    <xacro:property name="params" value="${xacro.load_yaml(yaml_param_file)}"/>
-<xacro:macro name="wheel" params="name prefix">
-        <joint name="${prefix}${name}_wheel_joint" type="continuous">
+  <xacro:property name="yaml_param_file" value="$(find mirte_base_control)/config/control_master.yaml"/>
+  <xacro:property name="params" value="${xacro.load_yaml(yaml_param_file)}"/>
+  <xacro:macro name="wheel" params="name prefix">
+    <joint name="${prefix}${name}_wheel_joint" type="fixed">
       <parent link="${prefix}base_link"/>
       <child link="${prefix}${name}_wheel"/>
@@ -11,45 +11,97 @@
       <axis xyz="0 1 0"/>
       <dynamics damping="0.2"/>
+      <pose>0 0 0 0 0 0</pose>
     </joint>
     <!-- left wheel Link -->
     <link name="${prefix}${name}_wheel">
 </link>
-</xacro:macro>
-<xacro:macro name="joint" params="name prefix">
-      <joint name="${prefix}${name}_wheel_joint">
-        <command_interface name="velocity"/>
-        <state_interface name="position"/>
-        <state_interface name="velocity"/>
-      </joint>
-</xacro:macro>
-  <xacro:arg name="prefix" default="" />
-    <link name="base_link">
+  </xacro:macro>
+  <xacro:macro name="joint" params="name prefix">
+    <joint name="${prefix}${name}_wheel_joint">
+      <command_interface name="velocity"/>
+      <state_interface name="position"/>
+      <state_interface name="velocity"/>
+    </joint>
+  </xacro:macro>
+  <xacro:arg name="prefix" default=""/>
+  <link name="base_link">
 </link>
-<!-- same ordering as the mecanum drive controller -->
-        <xacro:wheel name="left_front" prefix="$(arg prefix)" />
-        <xacro:wheel name="left_rear" prefix="$(arg prefix)" />
-        <xacro:wheel name="right_rear" prefix="$(arg prefix)" />
-        <xacro:wheel name="right_front" prefix="$(arg prefix)" />
-            <ros2_control name="mecanumdrive" type="system">
-      <hardware>
-        <plugin>mirte_base_control/MirteBaseHWInterface</plugin>
-        <param name="ticks">${params['ticks']}</param>
-        <param name="enable_pid">${params['enable_pid']}</param>
-        <param name="kp">${params['kp']}</param>
-        <param name="ki">${params['ki']}</param>
-        <param name="kd">${params['kd']}</param>
-        <param name="i_clamp">${params['i_clamp']}</param>
-        <param name="antiwindup">${params['antiwindup']}</param>
-      </hardware>
-      <xacro:joint prefix="$(arg prefix)" name="left_front"  />
-        <xacro:joint prefix="$(arg prefix)" name="right_front"  />
-        <xacro:joint prefix="$(arg prefix)" name="left_rear"  />
-        <xacro:joint prefix="$(arg prefix)" name="right_rear"  />
-      <!-- <joint name="${prefix}right_wheel_joint">
+  <!-- same ordering as the mecanum drive controller -->
+  <xacro:wheel name="left_front" prefix="$(arg prefix)"/>
+  <xacro:wheel name="left_rear" prefix="$(arg prefix)"/>
+  <xacro:wheel name="right_rear" prefix="$(arg prefix)"/>
+  <xacro:wheel name="right_front" prefix="$(arg prefix)"/>
+  <ros2_control name="mecanumdrive" type="system">
+    <hardware>
+      <plugin>mirte_base_control/MirteBaseHWInterface</plugin>
+      <param name="ticks">${params['ticks']}</param>
+      <param name="enable_pid">${params['enable_pid']}</param>
+      <param name="kp">${params['kp']}</param>
+      <param name="ki">${params['ki']}</param>
+      <param name="kd">${params['kd']}</param>
+      <param name="i_clamp">${params['i_clamp']}</param>
+      <param name="antiwindup">${params['antiwindup']}</param>
+    </hardware>
+    <xacro:joint prefix="$(arg prefix)" name="left_front"/>
+    <xacro:joint prefix="$(arg prefix)" name="right_front"/>
+    <xacro:joint prefix="$(arg prefix)" name="left_rear"/>
+    <xacro:joint prefix="$(arg prefix)" name="right_rear"/>
+    <!-- <joint name="${prefix}right_wheel_joint">
         <command_interface name="velocity"/>
         <state_interface name="position"/>
         <state_interface name="velocity"/>
       </joint> -->
-    </ros2_control>
+  </ros2_control>
+   <joint name="lidar" type="fixed">
+    <origin rpy="0 0 0" xyz="0.012 0 0.105"/>
+    <parent link="base_link"/>
+    <child link="lidar_link"/>
+  </joint>
+  <link name="lidar_link">
+    <visual>
+      <origin rpy="0 0 0" xyz="0 0 -0.03"/>
+      <geometry>
+        <mesh filename="file://$(find mirte_gazebo)/meshes/lidar.stl" scale="0.001 0.001 0.001" rpy="0 0 1.57079633"/>
+      </geometry>
+    </visual>
+    <collision>
+      <origin rpy="0 0 0" xyz="0 0 -0.03"/>
+      <geometry>
+        <mesh filename="file://$(find mirte_gazebo)/meshes/lidar.stl" scale="0.001 0.001 0.001" rpy="0 0 1.57079633"/>
+      </geometry>
+    </collision>
+  </link>
+  <gazebo reference="lidar_link">
+    <sensor name="lidar" type="ray">
+      <pose>0 0 0 0 0 0</pose>
+      <visualize>true</visualize>
+      <update_rate>10</update_rate>
+      <ray>
+        <scan>
+          <horizontal>
+            <samples>720</samples>
+            <resolution>1</resolution>
+            <min_angle>-3.14</min_angle>
+            <max_angle>3.14</max_angle>
+          </horizontal>
+        </scan>
+        <range>
+          <min>0.15</min>
+          <!-- bit more than the actual min range of the lidar, but otherwise it will detect the mirte itself-->
+          <max>12</max>
+          <resolution>0.01</resolution>
+        </range>
+        <noise>
+          <type>gaussian</type>
+          <mean>0.0</mean>
+          <stddev>0.01</stddev>
+        </noise>
+      </ray>
+      <plugin name="ultra_controller" filename="libgazebo_ros_laser.so">
+        <topicName>/mirte/scan</topicName>
+        <frameName>lidar_link</frameName>
+      </plugin>
+    </sensor>
+  </gazebo>
   <!-- <xacro:include filename="$(find mirte_control)/urdf/diffbot_description.urdf.xacro" />
   <!- -  Import Rviz colors - ->

File: mirte_control/description/ros2_control/diffbot.ros2_control.xacro (robot description, xacro)
@@ -7,12 +7,12 @@
       </hardware>
       <joint name="${prefix}left_wheel_joint">
-        <command_interface name="velocity" />
-        <state_interface name="position" />
-        <state_interface name="velocity" />
+        <command_interface name="velocity"/>
+        <state_interface name="position"/>
+        <state_interface name="velocity"/>
       </joint>
       <joint name="${prefix}right_wheel_joint">
-        <command_interface name="velocity" />
-        <state_interface name="position" />
-        <state_interface name="velocity" />
+        <command_interface name="velocity"/>
+        <state_interface name="position"/>
+        <state_interface name="velocity"/>
       </joint>
     </ros2_control>

File: mirte_control/description/urdf/diffbot.urdf.xacro (robot description, xacro)
@@ -2,12 +2,11 @@
 <!-- Basic differential drive mobile base -->
 <robot xmlns:xacro="http://www.ros.org/wiki/xacro" name="diffdrive_robot">
-  <xacro:arg name="prefix" default="" />
-  <xacro:include filename="$(find mirte_control)/urdf/diffbot_description.urdf.xacro" />
+  <xacro:arg name="prefix" default=""/>
+  <xacro:include filename="$(find mirte_control)/urdf/diffbot_description.urdf.xacro"/>
   <!-- Import Rviz colors -->
-  <xacro:include filename="$(find mirte_control)/urdf/diffbot.materials.xacro" />
+  <xacro:include filename="$(find mirte_control)/urdf/diffbot.materials.xacro"/>
   <!-- Import diffbot ros2_control description -->
-  <xacro:include filename="$(find mirte_control)/ros2_control/diffbot.ros2_control.xacro" />
-  <xacro:diffbot prefix="$(arg prefix)" />
-  <xacro:diffbot_ros2_control
-    name="MirteHardware" prefix="$(arg prefix)" />
+  <xacro:include filename="$(find mirte_control)/ros2_control/diffbot.ros2_control.xacro"/>
+  <xacro:diffbot prefix="$(arg prefix)"/>
+  <xacro:diffbot_ros2_control name="MirteHardware" prefix="$(arg prefix)"/>
 </robot>

File: mirte_control/description/urdf/diffbot_description.urdf.xacro (robot description, xacro)
@@ -2,38 +2,39 @@
 <robot xmlns:xacro="http://www.ros.org/wiki/xacro">
   <xacro:macro name="diffbot" params="prefix">
-  <!-- Constants for robot dimensions -->
-  <xacro:property name="PI" value="3.1415926535897931"/>
-  <xacro:property name="base_mass" value="0.3" /> <!-- arbitrary value for base mass -->
-  <xacro:property name="base_width" value="0.125" />
-  <xacro:property name="base_length" value="0.22" />
-  <xacro:property name="base_height" value="0.1" />
-  <xacro:property name="wheel_mass" value="0.3" /> <!-- arbitrary value for wheel mass -->
-  <xacro:property name="wheel_len" value="0.01" />
-  <xacro:property name="wheel_radius" value="0.003" />
-  <xacro:property name="caster_wheel_mass" value="0.1" /> <!-- arbitrary value for caster wheel mass -->
-  <xacro:property name="caster_wheel_radius" value="0.015" />
-  <xacro:property name="z_offset" value="-${base_height/2}" /> <!-- Space btw top of beam and the each joint -->
-  <!-- Base Link -->
-  <link name="${prefix}base_link">
-    <collision>
-      <origin xyz="0 0 0" rpy="0 0 0"/>
-      <geometry>
-        <box size="${base_width} ${base_length} ${base_height}"/>
-      </geometry>
-    </collision>
-    <visual>
-      <origin xyz="0 0 ${base_height/2}" rpy="0 0 0"/>
-      <geometry>
-        <box size="${base_width} ${base_length} ${base_height}"/>
-      </geometry>
-      <material name="orange"/>
-    </visual>
-    <inertial>
-      <origin xyz="0 0 0" rpy="0 0 0"/>
-      <mass value="${base_mass}"/>
-      <inertia
-        ixx="${base_mass / 12.0 * (base_length*base_length + base_height*base_height)}" ixy="0.0" ixz="0.0"
-        iyy="${base_mass / 12.0 * (base_height*base_height + base_width*base_width)}" iyz="0.0"
-        izz="${base_mass / 12.0 * (base_width*base_width + base_length*base_length)}"/>
+    <!-- Constants for robot dimensions -->
+    <xacro:property name="PI" value="3.1415926535897931"/>
+    <xacro:property name="base_mass" value="0.3"/>
+    <!-- arbitrary value for base mass -->
+    <xacro:property name="base_width" value="0.125"/>
+    <xacro:property name="base_length" value="0.22"/>
+    <xacro:property name="base_height" value="0.1"/>
+    <xacro:property name="wheel_mass" value="0.3"/>
+    <!-- arbitrary value for wheel mass -->
+    <xacro:property name="wheel_len" value="0.01"/>
+    <xacro:property name="wheel_radius" value="0.003"/>
+    <xacro:property name="caster_wheel_mass" value="0.1"/>
+    <!-- arbitrary value for caster wheel mass -->
+    <xacro:property name="caster_wheel_radius" value="0.015"/>
+    <xacro:property name="z_offset" value="-${base_height/2}"/>
+    <!-- Space btw top of beam and the each joint -->
+    <!-- Base Link -->
+    <link name="${prefix}base_link">
+      <collision>
+        <origin xyz="0 0 0" rpy="0 0 0"/>
+        <geometry>
+          <box size="${base_width} ${base_length} ${base_height}"/>
+        </geometry>
+      </collision>
+      <visual>
+        <origin xyz="0 0 ${base_height/2}" rpy="0 0 0"/>
+        <geometry>
+          <box size="${base_width} ${base_length} ${base_height}"/>
+        </geometry>
+        <material name="orange"/>
+      </visual>
+      <inertial>
+        <origin xyz="0 0 0" rpy="0 0 0"/>
+        <mass value="${base_mass}"/>
+        <inertia ixx="${base_mass / 12.0 * (base_length*base_length + base_height*base_height)}" ixy="0.0" ixz="0.0" iyy="${base_mass / 12.0 * (base_height*base_height + base_width*base_width)}" iyz="0.0" izz="${base_mass / 12.0 * (base_width*base_width + base_length*base_length)}"/>
       </inertial>
     </link>
@@ -63,10 +64,7 @@
         <origin xyz="0 0 0" rpy="${PI/2} 0 0"/>
         <mass value="${wheel_mass}"/>
-        <inertia
-          ixx="${wheel_mass / 12.0 * (3*wheel_radius + wheel_len*wheel_len)}" ixy="0.0" ixz="0.0"
-          iyy="${wheel_mass / 12.0 * wheel_radius*wheel_radius}" iyz="0.0"
-          izz="${wheel_mass / 12.0 * wheel_radius*wheel_radius}"/>
-        </inertial>
-      </link>
+        <inertia ixx="${wheel_mass / 12.0 * (3*wheel_radius + wheel_len*wheel_len)}" ixy="0.0" ixz="0.0" iyy="${wheel_mass / 12.0 * wheel_radius*wheel_radius}" iyz="0.0" izz="${wheel_mass / 12.0 * wheel_radius*wheel_radius}"/>
+      </inertial>
+    </link>
     <joint name="${prefix}right_wheel_joint" type="continuous">
       <parent link="${prefix}base_link"/>
@@ -94,10 +92,7 @@
         <origin xyz="0 0 0" rpy="${PI/2} 0 0"/>
         <mass value="${wheel_mass}"/>
-        <inertia
-          ixx="${wheel_mass / 12.0 * (3*wheel_radius + wheel_len*wheel_len)}" ixy="0.0" ixz="0.0"
-          iyy="${wheel_mass / 12.0 * wheel_radius*wheel_radius}" iyz="0.0"
-          izz="${wheel_mass / 12.0 * wheel_radius*wheel_radius}"/>
-        </inertial>
-      </link>
+        <inertia ixx="${wheel_mass / 12.0 * (3*wheel_radius + wheel_len*wheel_len)}" ixy="0.0" ixz="0.0" iyy="${wheel_mass / 12.0 * wheel_radius*wheel_radius}" iyz="0.0" izz="${wheel_mass / 12.0 * wheel_radius*wheel_radius}"/>
+      </inertial>
+    </link>
     <joint name="${prefix}caster_frontal_wheel_joint" type="fixed">
       <parent link="${prefix}base_link"/>
@@ -123,10 +118,7 @@
         <origin xyz="0 0 0" rpy="0 0 0"/>
         <mass value="${caster_wheel_mass}"/>
-        <inertia
-          ixx="${caster_wheel_mass * 0.4 * (caster_wheel_radius * caster_wheel_radius)}" ixy="0.0" ixz="0.0"
-          iyy="${caster_wheel_mass * 0.4 * (caster_wheel_radius * caster_wheel_radius)}" iyz="0.0"
-          izz="${caster_wheel_mass * 0.4 * (caster_wheel_radius * caster_wheel_radius)}"/>
-        </inertial>
-      </link>
+        <inertia ixx="${caster_wheel_mass * 0.4 * (caster_wheel_radius * caster_wheel_radius)}" ixy="0.0" ixz="0.0" iyy="${caster_wheel_mass * 0.4 * (caster_wheel_radius * caster_wheel_radius)}" iyz="0.0" izz="${caster_wheel_mass * 0.4 * (caster_wheel_radius * caster_wheel_radius)}"/>
+      </inertial>
+    </link>
     <joint name="${prefix}caster_rear_wheel_joint" type="fixed">
       <parent link="${prefix}base_link"/>
@@ -152,10 +144,7 @@
         <origin xyz="0 0 0" rpy="0 0 0"/>
         <mass value="${caster_wheel_mass}"/>
-        <inertia
-          ixx="${caster_wheel_mass * 0.4 * (caster_wheel_radius * caster_wheel_radius)}" ixy="0.0" ixz="0.0"
-          iyy="${caster_wheel_mass * 0.4 * (caster_wheel_radius * caster_wheel_radius)}" iyz="0.0"
-          izz="${caster_wheel_mass * 0.4 * (caster_wheel_radius * caster_wheel_radius)}"/>
-        </inertial>
-      </link>
+        <inertia ixx="${caster_wheel_mass * 0.4 * (caster_wheel_radius * caster_wheel_radius)}" ixy="0.0" ixz="0.0" iyy="${caster_wheel_mass * 0.4 * (caster_wheel_radius * caster_wheel_radius)}" iyz="0.0" izz="${caster_wheel_mass * 0.4 * (caster_wheel_radius * caster_wheel_radius)}"/>
+      </inertial>
+    </link>
   </xacro:macro>
 </robot>
