Commit message: start moveit ros2

File: mirte_control/mirte_master_arm_control/bringup/urdf/arm.urdf.xacro (robot description, xacro)
@@ -4,5 +4,5 @@
     <xacro:property name="yaml_param_file" value="$(find mirte_base_control)/config/control_master.yaml"/>
     <xacro:property name="params" value="${xacro.load_yaml(yaml_param_file)}"/>
- <link
+ <!-- <link
         name="arm_Rot">
         <inertial>
@@ -588,5 +588,5 @@
             effort="0"
             velocity="0" />
-    </joint>
+    </joint>-->
     <xacro:macro name="joint" params="name prefix">
       <joint name="arm_${prefix}${name}_joint">
@@ -610,8 +610,8 @@
         <param name="antiwindup">${params['antiwindup']}</param> -->
       </hardware>
-      <xacro:joint prefix="$(arg prefix)" name="rotate"  />
-        <xacro:joint prefix="$(arg prefix)" name="shoulder"  />
-        <xacro:joint prefix="$(arg prefix)" name="elbow"  />
-        <xacro:joint prefix="$(arg prefix)" name="wrist"  />
+      <xacro:joint prefix="$(arg prefix)" name="Rot"  />
+        <xacro:joint prefix="$(arg prefix)" name="Shoulder"  />
+        <xacro:joint prefix="$(arg prefix)" name="Elbow"  />
+        <xacro:joint prefix="$(arg prefix)" name="Wrist"  />
       <!-- <joint name="${prefix}right_wheel_joint">
         <command_interface name="velocity"/>

File: mirte_description/mirte_master_description/urdf/mirte_master.xacro (robot description, xacro)
@@ -10,4 +10,5 @@
   <xacro:arg name="depth_camera_enable" default="False" />
   <xacro:arg name="imu_enable" default="False" />
+  <xacro:arg name="use_gazebo" default="False" />
   <xacro:arg name="use_namespace" default="False"/>
   <xacro:arg name="namespace_name" default="" />

File: mirte_description/mirte_master_description/urdf/ros2_control.xacro (robot description, xacro)
@@ -1,4 +1,5 @@
 <?xml version="1.0"?>
 <robot xmlns:xacro="http://www.ros.org/wiki/xacro">
+<xacro:if value="$(arg use_gazebo)">
   <ros2_control name="GazeboSystem" type="system">
     <hardware>
@@ -62,4 +63,5 @@
     </joint>
   </ros2_control>
+</xacro:if>
 <gazebo>
     <plugin filename="libgazebo_ros2_control.so" name="gazebo_ros2_control">

File: mirte_master_moveit_config/config/mirte_master.ros2_control.xacro (robot description, xacro)
@@ -6,5 +6,5 @@
             <hardware>
                 <!-- By default, set up controllers for simulation. This won't work on real hardware -->
-                <plugin>mock_components/GenericSystem</plugin>
+                <plugin>mirte_master_arm_control/MirteMasterArmHWInterface</plugin>
             </hardware>
             <joint name="arm_Rot_joint">
@@ -32,10 +32,10 @@
                 </state_interface>
             </joint>
-            <joint name="Gripper_joint">
+            <!-- <joint name="Gripper_joint">
                 <command_interface name="position"/>
                 <state_interface name="position">
                   <param name="initial_value">${initial_positions['Gripper_joint']}</param>
                 </state_interface>
-            </joint>
+            </joint> -->
         </ros2_control>
     </xacro:macro>
