Commit message: bringup config moves

File: mirte_control/mirte_master_arm_control/bringup/urdf/arm.urdf.xacro (robot description, xacro)
@@ -2,6 +2,4 @@
 <!-- Basic differential drive mobile base -->
 <robot xmlns:xacro="http://www.ros.org/wiki/xacro" name="diffdrive_robot">
-    <xacro:property name="yaml_param_file" value="$(find mirte_base_control)/config/control_master.yaml"/>
-    <xacro:property name="params" value="${xacro.load_yaml(yaml_param_file)}"/>
  <link
         name="arm_Rot">
@@ -602,11 +600,4 @@
       <hardware>
         <plugin>mirte_master_arm_control/MirteMasterArmHWInterface</plugin>
-        <!-- <param name="ticks">${params['ticks']}</param>
-        <param name="enable_pid">${params['enable_pid']}</param>
-        <param name="kp">${params['kp']}</param>
-        <param name="ki">${params['ki']}</param>
-        <param name="kd">${params['kd']}</param>
-        <param name="i_clamp">${params['i_clamp']}</param>
-        <param name="antiwindup">${params['antiwindup']}</param> -->
       </hardware>
       <xacro:joint prefix="$(arg prefix)" name="rotate"  />
@@ -614,9 +605,4 @@
         <xacro:joint prefix="$(arg prefix)" name="elbow"  />
         <xacro:joint prefix="$(arg prefix)" name="wrist"  />
-      <!-- <joint name="${prefix}right_wheel_joint">
-        <command_interface name="velocity"/>
-        <state_interface name="position"/>
-        <state_interface name="velocity"/>
-      </joint> -->
     </ros2_control>
 </robot>
