Commit message: mmv2 desc: Add arm gripper cam

File: mirte_description/mirte_master_description/urdf/mirte_masterv2.xacro (robot description, xacro)
@@ -3,6 +3,17 @@
      Commit Version: 1.6.0-4-g7f85cfe  Build Version: 1.6.7995.38578
      For more information, please see http://wiki.ros.org/sw_urdf_exporter -->
-<robot
+<robot xmlns:xacro="http://www.ros.org/wiki/xacro"
   name="mirte_master_description">
+    <xacro:arg name="arm_enable" default="True" />
+    <xacro:arg name="enable_arm_collisions" default="True" />
+    <xacro:arg name="arm_camera_enable" default="True" />
+  <xacro:arg name="front_camera_enable" default="False" />
+  <xacro:arg name="sonar_enable" default="True" />
+  <xacro:arg name="lidar_enable" default="True" />
+  <xacro:arg name="depth_camera_enable" default="True" />
+  <xacro:arg name="imu_enable" default="True" />
+  <xacro:arg name="gripper_camera" default="True" />
+  <xacro:arg name="wheels_enable" default="True" />
+  <xacro:arg name="sim" default="False" />
   <link
     name="MIRTE_Master">
@@ -310,462 +321,8 @@
       xyz="0 -1 0" />
   </joint>
-  <link
-    name="Arm">
-    <inertial>
-      <origin
-        xyz="0.199878078588349 -0.00452321557552078 0.245475596940599"
-        rpy="0 0 0" />
-      <mass
-        value="0.438578226451647" />
-      <inertia
-        ixx="0.000220377694326858"
-        ixy="-1.48489357771068E-06"
-        ixz="-5.53821777263242E-05"
-        iyy="0.000249243731826793"
-        iyz="-3.26836277134958E-06"
-        izz="0.000214737746366638" />
-    </inertial>
-    <!-- <visual>
-      <origin
-        xyz="0 0 0"
-        rpy="0 0 0" />
-      <geometry>
-        <mesh
-          filename="package://mirte_master_description/meshes/Arm.STL" />
-      </geometry>
-      <material
-        name="">
-        <color
-          rgba="0.752941176470588 0.752941176470588 0.752941176470588 1" />
-      </material>
-    </visual>
-    <collision>
-      <origin
-        xyz="0 0 0"
-        rpy="0 0 0" />
-      <geometry>
-        <mesh
-          filename="package://mirte_master_description/meshes/Arm.STL" />
-      </geometry>
-    </collision> -->
-  </link>
-  <joint
-    name="Arm_joint"
-    type="fixed">
-    <origin
-      xyz="0.00012036 -0.01012 -0.0024812"
-      rpy="1.5708 0 0" />
-    <parent
-      link="MIRTE_Master" />
-    <child
-      link="Arm" />
-    <axis
-      xyz="0 0 0" />
-  </joint>
-  <link
-    name="z-Rotation">
-    <inertial>
-      <origin
-        xyz="-0.00543776553160195 -0.000509501501145752 0.0285808246077279"
-        rpy="0 0 0" />
-      <mass
-        value="0.0526781402686753" />
-      <inertia
-        ixx="1.27936978119511E-05"
-        ixy="2.24649358664918E-07"
-        ixz="3.24570783940582E-07"
-        iyy="9.0108967812021E-06"
-        iyz="3.19125827976664E-08"
-        izz="1.70619631994108E-05" />
-    </inertial>
-    <visual>
-      <origin
-        xyz="0 0 0"
-        rpy="0 0 0" />
-      <geometry>
-        <mesh
-          filename="package://mirte_master_description/meshes/z-Rotation.STL" />
-      </geometry>
-      <material
-        name="">
-        <color
-          rgba="0.752941176470588 0.752941176470588 0.752941176470588 1" />
-      </material>
-    </visual>
-    <collision>
-      <origin
-        xyz="0 0 0"
-        rpy="0 0 0" />
-      <geometry>
-        <mesh
-          filename="package://mirte_master_description/meshes/z-Rotation.STL" />
-      </geometry>
-    </collision>
-  </link>
-  <joint
-    name="z-Rotation_joint"
-    type="continuous">
-    <origin
-      xyz="0.121551322610448 -0.00891627722041789 0.110848128389983"
-      rpy="0 2.66843023091516E-05 0" />
-    <parent
-      link="Arm" />
-    <child
-      link="z-Rotation" />
-    <axis
-      xyz="0 0 1" />
-    <limit
-      lower="0"
-      upper="0"
-      effort="0"
-      velocity="0" />
-  </joint>
-  <link
-    name="Upperarm">
-    <inertial>
-      <origin
-        xyz="0.0243247540835085 -0.0302970421840243 0.0844721417436619"
-        rpy="0 0 0" />
-      <mass
-        value="0.102325054139096" />
-      <inertia
-        ixx="0.000110625274617278"
-        ixy="8.06428564589689E-07"
-        ixz="-2.1315067607945E-05"
-        iyy="9.74019221425693E-05"
-        iyz="-1.18220607812138E-06"
-        izz="3.61861144527713E-05" />
-    </inertial>
-    <visual>
-      <origin
-        xyz="0 0 0"
-        rpy="0 0 0" />
-      <geometry>
-        <mesh
-          filename="package://mirte_master_description/meshes/Upperarm.STL" />
-      </geometry>
-      <material
-        name="">
-        <color
-          rgba="0.752941176470588 0.752941176470588 0.752941176470588 1" />
-      </material>
-    </visual>
-    <collision>
-      <origin
-        xyz="0 0 0"
-        rpy="0 0 0" />
-      <geometry>
-        <mesh
-          filename="package://mirte_master_description/meshes/Upperarm.STL" />
-      </geometry>
-    </collision>
-  </link>
-  <joint
-    name="Shoulder_joint"
-    type="continuous">
-    <origin
-      xyz="0.00380301601043069 0.0313794450114005 0.0332500000000377"
-      rpy="0 -2.66843023091516E-05 0" />
-    <parent
-      link="z-Rotation" />
-    <child
-      link="Upperarm" />
-    <axis
-      xyz="-0.0590713107277822 0.998253765455667 0" />
-    <limit
-      lower="0"
-      upper="0"
-      effort="0"
-      velocity="0" />
-  </joint>
-  <link
-    name="Forearm">
-    <inertial>
-      <origin
-        xyz="0.0706772608618316 -0.027444951764167 0.0395073033756355"
-        rpy="0 0 0" />
-      <mass
-        value="0.0911215389802598" />
-      <inertia
-        ixx="4.06272465991904E-05"
-        ixy="-2.95497241375996E-06"
-        ixz="-3.39941318616991E-05"
-        iyy="9.04576214125665E-05"
-        iyz="-2.00928077391389E-06"
-        izz="8.03522239189564E-05" />
-    </inertial>
-    <visual>
-      <origin
-        xyz="0 0 0"
-        rpy="0 0 0" />
-      <geometry>
-        <mesh
-          filename="package://mirte_master_description/meshes/Forearm.STL" />
-      </geometry>
-      <material
-        name="">
-        <color
-          rgba="0.752941176470588 0.752941176470588 0.752941176470588 1" />
-      </material>
-    </visual>
-    <collision>
-      <origin
-        xyz="0 0 0"
-        rpy="0 0 0" />
-      <geometry>
-        <mesh
-          filename="package://mirte_master_description/meshes/Forearm.STL" />
-      </geometry>
-    </collision>
-  </link>
-  <joint
-    name="Elbow_joint"
-    type="continuous">
-    <origin
-      xyz="0.036437928080887 0.00180537281653873 0.137006236814825"
-      rpy="0 0 0" />
-    <parent
-      link="Upperarm" />
-    <child
-      link="Forearm" />
-    <axis
-      xyz="-0.0590713107275747 0.998253765455679 0" />
-    <limit
-      lower="0"
-      upper="0"
-      effort="0"
-      velocity="0" />
-  </joint>
-  <link
-    name="Wrist">
-    <inertial>
-      <origin
-        xyz="0.030457565932454 -0.0213199330141271 0.0246561263482211"
-        rpy="0 0 0" />
-      <mass
-        value="0.0631657082718983" />
-      <inertia
-        ixx="1.94207147453815E-05"
-        ixy="3.79658302272387E-07"
-        ixz="9.22730385151376E-07"
-        iyy="1.35649196766237E-05"
-        iyz="6.81817829335488E-08"
-        izz="1.75049753123464E-05" />
-    </inertial>
-    <visual>
-      <origin
-        xyz="0 0 0"
-        rpy="0 0 0" />
-      <geometry>
-        <mesh
-          filename="package://mirte_master_description/meshes/Wrist.STL" />
-      </geometry>
-      <material
-        name="">
-        <color
-          rgba="0.752941176470588 0.752941176470588 0.752941176470588 1" />
-      </material>
-    </visual>
-    <collision>
-      <origin
-        xyz="0 0 0"
-        rpy="0 0 0" />
-      <geometry>
-        <mesh
-          filename="package://mirte_master_description/meshes/Wrist.STL" />
-      </geometry>
-    </collision>
-  </link>
-  <joint
-    name="Wrist_joint"
-    type="continuous">
-    <origin
-      xyz="0.124425999226755 0.000550856546668227 0.0712063710175444"
-      rpy="0 0 0" />
-    <parent
-      link="Forearm" />
-    <child
-      link="Wrist" />
-    <axis
-      xyz="-0.0590713107276118 0.998253765455677 0" />
-    <limit
-      lower="0"
-      upper="0"
-      effort="0"
-      velocity="0" />
-  </joint>
-  <link
-    name="Gripper_Left">
-    <inertial>
-      <origin
-        xyz="0.0260104638193439 0.0194222325489568 0.0221346361100294"
-        rpy="0 0 0" />
-      <mass
-        value="0.0189805948365668" />
-      <inertia
-        ixx="2.34101098127276E-06"
-        ixy="3.22622491333076E-07"
-        ixz="-8.17376363293455E-07"
-        iyy="2.49216095826188E-06"
-        iyz="1.86856580622951E-07"
-        izz="3.84236227432968E-06" />
-    </inertial>
-    <visual>
-      <origin
-        xyz="0 0 0"
-        rpy="0 0 0" />
-      <geometry>
-        <mesh
-          filename="package://mirte_master_description/meshes/Gripper_Left.STL" />
-      </geometry>
-      <material
-        name="">
-        <color
-          rgba="0.752941176470588 0.752941176470588 0.752941176470588 1" />
-      </material>
-    </visual>
-    <collision>
-      <origin
-        xyz="0 0 0"
-        rpy="0 0 0" />
-      <geometry>
-        <mesh
-          filename="package://mirte_master_description/meshes/Gripper_Left.STL" />
-      </geometry>
-    </collision>
-  </link>
-  <joint
-    name="Left_gripper_joint"
-    type="continuous">
-    <origin
-      xyz="0.0505382985096727 -0.00913040976600391 0.006318005818223"
-      rpy="0 0 0" />
-    <parent
-      link="Wrist" />
-    <child
-      link="Gripper_Left" />
-    <axis
-      xyz="-0.384044127181366 -0.0226909681284593 0.923035875978229" />
-    <limit
-      lower="0"
-      upper="0"
-      effort="0"
-      velocity="0" />
-  </joint>
-  <link
-    name="Gripper_Right">
-    <inertial>
-      <origin
-        xyz="0.0251469938866446 -0.0152950047655913 0.0215607980324168"
-        rpy="0 0 0" />
-      <mass
-        value="0.020696726381591" />
-      <inertia
-        ixx="2.64854872929009E-06"
-        ixy="-2.65371466970767E-07"
-        ixz="-7.63828524600313E-07"
-        iyy="2.57591088627407E-06"
-        iyz="-3.63820979056845E-07"
-        izz="4.07757485928383E-06" />
-    </inertial>
-    <visual>
-      <origin
-        xyz="0 0 0"
-        rpy="0 0 0" />
-      <geometry>
-        <mesh
-          filename="package://mirte_master_description/meshes/Gripper_Right.STL" />
-      </geometry>
-      <material
-        name="">
-        <color
-          rgba="0.752941176470588 0.752941176470588 0.752941176470588 1" />
-      </material>
-    </visual>
-    <collision>
-      <origin
-        xyz="0 0 0"
-        rpy="0 0 0" />
-      <geometry>
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
Commit message: mmv2 desc: Add sonar

File: mirte_description/mirte_master_description/urdf/mirte_masterv2.xacro (robot description, xacro)
@@ -379,110 +379,39 @@
     <xacro:include filename="$(find mirte_master_description)/urdf/depth_cam.xacro" />
   </xacro:if>
-  <link
-    name="Sonar_left">
-    <inertial>
-      <origin
-        xyz="-0.00912435116484579 6.97371721982212E-05 0.0128430743123096"
-        rpy="0 0 0" />
-      <mass
-        value="0.00383513951999242" />
-      <inertia
-        ixx="7.68751523460338E-07"
-        ixy="-2.65063614506786E-09"
-        ixz="8.54213890540522E-10"
-        iyy="7.2622124271108E-07"
-        iyz="-3.40126465277456E-09"
-        izz="1.59365535001317E-07" />
-    </inertial>
-    <!-- <visual>
-      <origin
-        xyz="0 0 0"
-        rpy="0 0 0" />
-      <geometry>
-        <mesh
-          filename="package://mirte_master_description/meshes/Sonar_left.STL" />
-      </geometry>
-      <material
-        name="">
-        <color
-          rgba="0.792156862745098 0.819607843137255 0.933333333333333 1" />
-      </material>
-    </visual>
-    <collision>
-      <origin
-        xyz="0 0 0"
-        rpy="0 0 0" />
-      <geometry>
-        <mesh
-          filename="package://mirte_master_description/meshes/Sonar_left.STL" />
-      </geometry>
-    </collision> -->
-  </link>
-  <joint
-    name="Sonar_left_joint"
-    type="fixed">
-    <origin
-      xyz="-0.10657 -0.0059239 0.071178"
+  <xacro:if value="$(arg sonar_enable)">
+    <xacro:include filename="$(find mirte_master_description)/urdf/ultrasonic.xacro" />
+    <joint name="chassis_base_joint" type="fixed">
+      <parent link="Base" />
+      <child link="link_chassis" />
+    </joint>
+    <link name="link_chassis" />
+    <!-- <xacro:ultrasonic_sensor name="front_left">
+      <origin
+        xyz="0.05297775289576 -0.120282421780502 -0.031"
+        rpy="0 0 ${-pi/2+0.296705972839036}" />
+    </xacro:ultrasonic_sensor>
+    <xacro:ultrasonic_sensor name="front_right">
+      <origin
+        xyz="-0.05297775289576 -0.120282421780502 -0.031"
+        rpy="0 0 ${-pi/2-0.296705972839036}" />
+    </xacro:ultrasonic_sensor> -->
+    <xacro:ultrasonic_sensor name="rear_left">
+    <origin
+      xyz="-0.10657 -0.0209239 0.071178"
       rpy="-1.5708 -0.54098 -3.1416" />
-    <parent
-      link="Base" />
-    <child
-      link="Sonar_left" />
-    <axis
-      xyz="0 0 0" />
-  </joint>
-  <link
-    name="Sonar_right">
-    <inertial>
-      <origin
-        xyz="-0.00912435116482696 -6.99136580070495E-05 0.0127569266473762"
-        rpy="0 0 0" />
-      <mass
-        value="0.00383513951999247" />
-      <inertia
-        ixx="7.68751523460339E-07"
-        ixy="2.65062440645516E-09"
-        ixz="-8.54250314742505E-10"
-        iyy="7.2622114912563E-07"
-        iyz="-3.40905422018215E-09"
-        izz="1.59365628586768E-07" />
-    </inertial>
-    <!-- <visual>
-      <origin
-        xyz="0 0 0"
-        rpy="0 0 0" />
-      <geometry>
-        <mesh
-          filename="package://mirte_master_description/meshes/Sonar_right.STL" />
-      </geometry>
-      <material
-        name="">
-        <color
-          rgba="0.792156862745098 0.819607843137255 0.933333333333333 1" />
-      </material>
-    </visual>
-    <collision>
-      <origin
-        xyz="0 0 0"
-        rpy="0 0 0" />
-      <geometry>
-        <mesh
-          filename="package://mirte_master_description/meshes/Sonar_right.STL" />
-      </geometry>
-    </collision> -->
-  </link>
-  <joint
-    name="Sonar_right_joint"
-    type="fixed">
+      <!-- <origin
+        xyz="0.0565606470918482 0.119187021096338 -0.031"
+        rpy="0 0 ${-pi/2 + 2.84488668075076}" /> -->
+    </xacro:ultrasonic_sensor>
+    <xacro:ultrasonic_sensor name="rear_right">
+    <!-- TODO: check rotation of sonars -->
     <origin
       xyz="-0.10657 -0.0059239 -0.093973"
       rpy="-1.5708 0.54098 -3.1416" />
-    <parent
-      link="Base" />
-    <child
-      link="Sonar_right" />
-    <axis
-      xyz="0 0 0" />
-  </joint>
+      <!-- <origin
+        xyz="-0.0565606470918482 0.119187021096338 -0.031"
+        rpy="0 0 ${-pi/2 -2.84488668075076}" /> -->
+    </xacro:ultrasonic_sensor>
+  </xacro:if>
   <link
     name="LiDar">

Commit message: mmv2 desc: wheels fixed

File: mirte_description/mirte_master_description/urdf/mirte_masterv2.xacro (robot description, xacro)
@@ -15,4 +15,5 @@
     <xacro:arg name="arm_collisions_enable" default="True" />
     <xacro:arg name="gripper_camera_enable" default="True" />
+  <!-- <xacro:include filename="$(find mirte_master_description)/urdf/ros2_control.xacro"/>   -->
   <link
     name="MIRTE_Master">
@@ -55,5 +56,26 @@
     </collision> -->
   </link>
-  <link
+<xacro:if value="$(arg wheels_enable)">
+  <xacro:property name="wheel_radius" value="0.050" />
+  <xacro:property name="wheel_length" value="0.055" />
+  <xacro:property name="wheel_mass" value="2.15" />
+  <xacro:property name="wheel_velocity" value="8" />
+  <xacro:property name="wheel_effort" value="5" />
+  <xacro:include filename="$(find mirte_master_description)/urdf/wheel.xacro" />
+   <!-- 0.025   -1 -->
+  <joint
+    name="Wheels_joint"
+    type="fixed">
+    <origin
+      xyz="0.0316698713027512 -0.052970257715017 -0.0113974879084128"
+      rpy="1.5707963267949 0 2.66843002434429E-05" />
+    <parent
+      link="MIRTE_Master" />
+    <child
+      link="Wheels" />
+    <axis
+      xyz="0 0 0" />
+  </joint>
+   <link
     name="Wheels">
     <inertial>
@@ -71,4 +93,95 @@
         izz="0.000322183176907626" />
     </inertial>
+    <!-- <visual>
+      <origin
+        xyz="0 0 0"
+        rpy="0 0 0" />
+      <geometry>
+        <mesh
+          filename="package://mirte_master_description/meshes/Wheels.STL" />
+      </geometry>
+      <material
+        name="">
+        <color
+          rgba="0.792156862745098 0.819607843137255 0.933333333333333 1" />
+      </material>
+    </visual> -->
+    <collision>
+      <origin
+        xyz="0 0 0"
+        rpy="0 0 0" />
+      <!-- <geometry>
+        <mesh
+          filename="package://mirte_master_description/meshes/Wheels.STL" />
+      </geometry> -->
+    </collision>
+  </link>
+  <!-- <joint
+    name="Wheels_joint"
+    type="fixed">
+    <origin
+      xyz="0.0316698713027512 -0.052970257715017 -0.0113974879084128"
+      rpy="1.5707963267949 0 2.66843002434429E-05" />
+    <parent
+      link="MIRTE_Master" />
+    <child
+      link="Wheels" />
+    <axis
+      xyz="0 0 0" />
+  </joint> -->
+    <xacro:mecanum_wheel name="front_left" wheel_type="left" link_origin="0.0">
+      <!-- <origin
+        xyz="${0.153 - 0} -0.085 -0.0455"
+        rpy="1.5708 0 -1.5708" /> -->
+        <!-- 0.080503 0.1575 -0.063 -->
+        <origin
+        xyz="0.080503 0.1075 -0.063"
+        rpy="0 0 0" />
+    </xacro:mecanum_wheel>
+   <!-- 0.025   -1 -->
+    <!-- <xacro:mecanum_wheel name="rear_left" wheel_type="right" link_origin="0.025">
+      <origin
+        xyz="-0.080503 0.1075 -0.063"
+        rpy="1.5708 0 -1.5708" />
+    </xacro:mecanum_wheel> -->
+   <!-- -0.025   -1 -->
+    <xacro:mecanum_wheel name="front_right" wheel_type="right" link_origin="0">
+            <origin
+        xyz="0.080503 ${-0.1075-0.05} -0.063"
+        rpy="0 0 ${-pi}"/>
+<!--
+      <origin
+        xyz="${-0.153 + wheel_length} -0.085 -0.0455"
+        rpy="1.5708 0 -1.5708" /> -->
+    </xacro:mecanum_wheel>
+   <!-- -0.025   -1 -->
+    <xacro:mecanum_wheel name="rear_right" wheel_type="left" link_origin="0">
+            <origin
+        xyz="-0.080503 -0.1075 -0.063"
+        rpy="0 0 ${-pi}"/>
+    </xacro:mecanum_wheel>
+    <xacro:mecanum_wheel name="rear_left" wheel_type="right" link_origin="0">
+            <origin
+        xyz="-0.080503 ${0.1075+0.05} -0.063"
+        rpy="0 0 0"/>
+    </xacro:mecanum_wheel>
+</xacro:if>
+  <xacro:if value="false">
+  <link
+    name="Wheels">
+    <inertial>
+      <origin
+        xyz="-1.48511945796681E-10 1.64047594952699E-12 -0.0630000002157284"
+        rpy="0 0 0" />
+      <mass
+        value="1.06645993257182" />
+      <inertia
+        ixx="0.000322183176884843"
+        ixy="-3.32280220325118E-11"
+        ixz="8.60065297084518E-15"
+        iyy="0.000372782415195671"
+        iyz="1.24669808687478E-13"
+        izz="0.000322183176907626" />
+    </inertial>
     <visual>
       <origin
@@ -320,4 +433,5 @@
       xyz="0 -1 0" />
   </joint>
+</xacro:if>
   <xacro:if value="$(arg arm_enable)">
     <xacro:include filename="$(find mirte_master_description)/urdf/arm2.xacro" />
