Commit message: mmv2 desc: wheels

File: mirte_description/mirte_master_description/urdf/mirte_masterv2.xacro (robot description, xacro)
@@ -130,5 +130,5 @@
       xyz="0 0 0" />
   </joint> -->
-    <xacro:mecanum_wheel name="front_left" wheel_type="left" link_origin="0.0">
+    <xacro:mecanum_wheel name="front_left" wheel_type="left" link_origin="0.025">
       <!-- <origin
         xyz="${0.153 - 0} -0.085 -0.0455"
@@ -146,9 +146,9 @@
     </xacro:mecanum_wheel> -->
    <!-- -0.025   -1 -->
-    <xacro:mecanum_wheel name="front_right" wheel_type="right" link_origin="0">
+    <xacro:mecanum_wheel name="front_right" wheel_type="right" link_origin="-0.025">
             <origin
-        xyz="0.080503 ${-0.1075-0.05} -0.063"
-        rpy="0 0 ${-pi}"/>
-<!--
+        xyz="0.080503 ${-0.1075} -0.063"
+        rpy="0 0 0"/>
+<!-- pi
       <origin
         xyz="${-0.153 + wheel_length} -0.085 -0.0455"
@@ -156,10 +156,11 @@
     </xacro:mecanum_wheel>
    <!-- -0.025   -1 -->
-    <xacro:mecanum_wheel name="rear_right" wheel_type="left" link_origin="0">
+    <xacro:mecanum_wheel name="rear_right" wheel_type="left" link_origin="0.025">
             <origin
-        xyz="-0.080503 -0.1075 -0.063"
-        rpy="0 0 ${-pi}"/>
+        xyz="-0.080503 ${-0.1075-0.05} -0.063"
+        rpy="0 0 0"/>
+        <!-- pi -->
     </xacro:mecanum_wheel>
-    <xacro:mecanum_wheel name="rear_left" wheel_type="right" link_origin="0">
+    <xacro:mecanum_wheel name="rear_left" wheel_type="right" link_origin="-0.025">
             <origin
         xyz="-0.080503 ${0.1075+0.05} -0.063"

File: mirte_description/mirte_master_description/urdf/ros2_control.xacro (robot description, xacro)
@@ -130,8 +130,21 @@
        </xacro:if>
     </plugin>
-    <plugin filename="libgazebo_ros_planar_move.so" name="gazebo_planar_move">
-       <robot_base_frame>base_link</robot_base_frame>
-    </plugin>
-    <plugin name="libgazebo_ros_p3d" filename="libgazebo_ros_p3d.so">
+     <!-- <plugin filename="gz-sim-planar-move-system" name="gz::sim::systems::PlanarMove">
+       <link_name>Base</link_name>
+     </plugin> -->
+     <plugin filename="gz-sim-mecanum-drive-system" name="gz::sim::systems::MecanumDrive">
+       <front_left_joint>front_left_wheel_joint</front_left_joint>
+       <front_right_joint>front_right_wheel_joint</front_right_joint>
+       <back_left_joint>rear_left_wheel_joint</back_left_joint>
+       <back_right_joint>rear_right_wheel_joint</back_right_joint>
+       <wheel_separation>0.28</wheel_separation>
+       <wheelbase>0.28</wheelbase>
+       <wheel_radius>0.05</wheel_radius>
+       <topic>cmd_vel</topic>
+       <odom_topic>odom</odom_topic>
+       <frame_id>odom</frame_id>
+       <child_frame_id>base_link</child_frame_id>
+     </plugin>
+    <!-- <plugin name="libgazebo_ros_p3d" filename="libgazebo_ros_p3d.so">
         <ros>
             <namespace>groundtruth</namespace>
@@ -142,5 +155,17 @@
         <update_rate>200.0</update_rate>
         <gaussian_noise>0.0</gaussian_noise>
-     </plugin>
+     </plugin> -->
+ <!-- <gazebo> -->
+  <plugin
+    filename="gz-sim-pose-publisher-system"
+    name="gz::sim::systems::PosePublisher">
+    <publish_link_pose>false</publish_link_pose>
+    <publish_collision_pose>false</publish_collision_pose>
+    <publish_visual_pose>false</publish_visual_pose>
+    <publish_nested_model_pose>false</publish_nested_model_pose>
+    <publish_model_pose>true</publish_model_pose>
+    <update_frequency>1</update_frequency>
+  </plugin>
+  <!-- </gazebo> -->
 </gazebo>
 </robot>

File: mirte_description/mirte_master_description/urdf/wheel.xacro (robot description, xacro)
@@ -2,5 +2,5 @@
 <!-- Copied from github:ArendJan/mirte-gazebo branch rsp -->
 <!-- Modified to remove the collision and change the minimum distance -->
-<robot xmlns:xacro="http://www.ros.org/wiki/xacro">
+<robot xmlns:xacro="http://www.ros.org/wiki/xacro" xmlns:gz="http://gazebosim.org/schema">
   <xacro:macro name="mecanum_wheel" params="name *origin link_origin wheel_type">
   <link
@@ -31,8 +31,24 @@
     </visual>
     <collision>
-      <origin xyz="0 0 ${link_origin}" />
+      <origin xyz="0 ${link_origin} 0" rpy="${pi/2} 0 0" />
       <geometry>
         <cylinder radius="${wheel_radius}" length="${wheel_length}" />
       </geometry>
+      <surface>
+            <friction>
+              <ode>
+                <mu>1.0</mu>
+                <mu2>0.0</mu2>
+                <xacro:if value="${wheel_type == 'left'}">
+                  <fdir1 gz:expressed_in="Wheels">-1 -1 0</fdir1>
+                </xacro:if>
+                <xacro:if value="${wheel_type == 'right'}">
+                  <fdir1 gz:expressed_in="Wheels">1 1 0</fdir1>
+                </xacro:if>
+                <!-- <fdir1 gz:expressed_in="Base">1 -1 0</fdir1> -->
+                                <!-- <fdir1 gz:expressed_in="chassis">1 -1 0</fdir1> -->
+              </ode>
+            </friction>
+          </surface>
     </collision>
   </link>
@@ -43,5 +59,5 @@
     <parent link="Wheels" />
     <child link="${name}_wheel" />
-    <axis xyz="0 -1 0" />
+    <axis xyz="0 1 0" />
   </joint>
   <transmission name="${name}_wheel_transmission">
