Commit message: mmv2 description start

File: mirte_description/mirte_master_description/urdf/depth_cam.xacro (robot description, xacro)
@@ -1,16 +1,17 @@
 <?xml version="1.0"?>
-<robot name="sensor_orbbec_astra_pro_plus" xmlns:xacro="http://ros.org/wiki/xacro">
-     <xacro:property name="orbbec_astra_pro_plus_scale" value="1.0" />
+<!-- uses new type depth cam, not astra pro plus, but astra mini pro. No stl for the camera as it's hidden in base frame -->
+<robot name="sensor_orbbec_astra_mini_pro" xmlns:xacro="http://ros.org/wiki/xacro">
+     <xacro:property name="orbbec_astra_mini_pro_scale" value="1.0" />
      <!-- RGB sensor - cam -->
      <!-- THESE MIGHT NEED TO CHANGE IF THE RESOLUTION IS NOT 640x480 -->
-     <xacro:property name="orbbec_astra_pro_plus_rel_rgb_px" value="0.0" />
-     <xacro:property name="orbbec_astra_pro_plus_rel_rgb_py" value="-0.0125" />
-     <xacro:property name="orbbec_astra_pro_plus_rel_rgb_pz" value="-0.0150" />
+     <xacro:property name="orbbec_astra_mini_pro_rel_rgb_px" value="0.0" />
+     <xacro:property name="orbbec_astra_mini_pro_rel_rgb_py" value="-0.0125" />
+     <xacro:property name="orbbec_astra_mini_pro_rel_rgb_pz" value="-0.0150" />
      <!-- IR sensor - depth -->
-     <xacro:property name="orbbec_astra_pro_plus_depth_rel_rgb_px" value="0.0" />
-     <xacro:property name="orbbec_astra_pro_plus_depth_rel_rgb_py" value="0.0250" />
-     <xacro:property name="orbbec_astra_pro_plus_depth_rel_rgb_pz" value="0.0" />
+     <xacro:property name="orbbec_astra_mini_pro_depth_rel_rgb_px" value="0.0" />
+     <xacro:property name="orbbec_astra_mini_pro_depth_rel_rgb_py" value="0.0250" />
+     <xacro:property name="orbbec_astra_mini_pro_depth_rel_rgb_pz" value="0.0" />
      <xacro:property name="M_PI" value="3.1415926535897931" />
-     <xacro:macro name="sensor_orbbec_astra_pro_plus"
+     <xacro:macro name="sensor_orbbec_astra_mini_pro"
           params="name parent *origin color rgb_w:=640 rgb_h:=480 stddev:=0.5">
           <joint name="${name}_rgb_joint" type="fixed">
@@ -40,5 +41,5 @@
           <joint name="${name}_joint" type="fixed">
                <origin
-                    xyz="${orbbec_astra_pro_plus_rel_rgb_px} ${orbbec_astra_pro_plus_rel_rgb_py} ${orbbec_astra_pro_plus_rel_rgb_pz}"
+                    xyz="${orbbec_astra_mini_pro_rel_rgb_px} ${orbbec_astra_mini_pro_rel_rgb_py} ${orbbec_astra_mini_pro_rel_rgb_pz}"
                     rpy="0.0 0 0" />
                <parent link="${name}_rgb_frame" />
@@ -69,5 +70,5 @@
           <joint name="${name}_depth_joint" type="fixed">
                <origin
-                    xyz="${orbbec_astra_pro_plus_depth_rel_rgb_px} ${orbbec_astra_pro_plus_depth_rel_rgb_py} ${orbbec_astra_pro_plus_depth_rel_rgb_pz}"
+                    xyz="${orbbec_astra_mini_pro_depth_rel_rgb_px} ${orbbec_astra_mini_pro_depth_rel_rgb_py} ${orbbec_astra_mini_pro_depth_rel_rgb_pz}"
                     rpy="0 0 0" />
                <parent link="${name}_rgb_frame" />
@@ -94,10 +95,10 @@
           </link>
           <!-- RGBD sensor for simulation, same as Kinect -->
-          <xacro:sensor_orbbec_astra_pro_plus_gazebo />
+          <xacro:sensor_orbbec_astra_mini_pro_gazebo />
      </xacro:macro>
      <!-- ====================================================
                            Gazebo
      ========================================================= -->
-     <xacro:macro name="sensor_orbbec_astra_pro_plus_gazebo">
+     <xacro:macro name="sensor_orbbec_astra_mini_pro_gazebo">
           <gazebo reference="${name}_link">
              <sensor name="${name}" type="depth">

File: mirte_description/mirte_master_description/urdf/mirte_master.xacro (robot description, xacro)
@@ -2,7 +2,5 @@
 <robot
   name="mirte_master" xmlns:xacro="http://ros.org/wiki/xacro">
-  <xacro:arg name="flag_enable" default="False" />
   <xacro:arg name="arm_enable" default="True" />
-  <xacro:arg name="screen_enable" default="False" />
   <xacro:arg name="front_camera_enable" default="False" />
   <xacro:arg name="sonar_enable" default="True" />
@@ -10,4 +8,6 @@
   <xacro:arg name="depth_camera_enable" default="True" />
   <xacro:arg name="imu_enable" default="True" />
+  <xacro:arg name="gripper_camera" default="True" />
+  <xacro:arg name="wheels_enable" default="True" />
   <xacro:arg name="sim" default="False" />
   <xacro:property name="camera_name" value="camera" lazy_eval="False"/>
@@ -27,8 +27,8 @@
   <xacro:include filename="$(find mirte_master_description)/urdf/mirte_master_base.gazebo.xacro" />
   <xacro:if value="$(arg depth_camera_enable)">
-    <xacro:include filename="$(find mirte_master_description)/urdf/orbbec_astra_plus_pro.xacro" />
-    <xacro:sensor_orbbec_astra_pro_plus name="${camera_name}" parent="frame_link" color="blue">
+    <xacro:include filename="$(find mirte_master_description)/urdf/depth_cam.xacro" />
+    <xacro:sensor_orbbec_astra_mini_pro name="${camera_name}" parent="frame_link" color="blue">
       <origin xyz="0.01 -0.146658788505756 0.0427" rpy="0 0 ${radians(-90)}" />
-    </xacro:sensor_orbbec_astra_pro_plus>
+    </xacro:sensor_orbbec_astra_mini_pro>
   </xacro:if>
   <xacro:if value="$(arg imu_enable)">
@@ -45,5 +45,5 @@
   </gazebo>
   <joint name="frame_base_joint" type="fixed">
-    <origin xyz="0 0 0.10" rpy="0 0 ${radians(90)}" />
+    <origin xyz="0 0 0.10" rpy="0 0 0" />
     <parent link="base_link" />
     <child link="frame_link" />
@@ -51,17 +51,27 @@
   <link
     name="frame_link">
-    <inertial>
-      <origin xyz="-0.00024285 0.0082178 ${-0.0037661 - 0.04}" />
-      <mass value="${base_mass}" />
+    <!-- <inertial> -->
+      <!-- <origin xyz="0.0344310118221643 -0.0286648891259541 -0.0113871267936065"/> -->
+      <!-- <mass value="${base_mass}" /> -->
+     <inertial>
+      <origin
+        xyz="0.0560559787388138 -0.046464113006352 -0.0107223863938312"
+        rpy="0 0 0" />
+      <mass
+        value="2.87187694310402" />
       <inertia
-        ixx="${base_mass * (0.06**2 + 0.28**2) / 12}"
-        iyy="${base_mass * (0.19**2 + 0.06**2) / 12}"
-        izz="${base_mass * (0.19**2 + 0.28**2) / 12}"
-        ixy="0" ixz="0" iyz="0" />
+        ixx="0.00268778032094885"
+        ixy="5.35777394513109E-05"
+        ixz="-1.34925830248996E-06"
+        iyy="0.006197833679705"
+        iyz="3.08873367085267E-06"
+        izz="0.00472317803422592" />
     </inertial>
-    <visual>
+    <visual> <origin
+        xyz="0 0 0"
+        rpy="0 0 0" />
       <geometry>
         <mesh
-          filename="package://mirte_master_description/meshes/frame_link.STL" />
+          filename="package://mirte_master_description/meshes/Base.STL" />
       </geometry>
       <material name="">
@@ -70,6 +80,7 @@
     </visual>
     <collision>
-      <origin xyz="0 0 -0.03" />
-      <geometry>
+  <origin
+        xyz="0 0 0"
+        rpy="0 0 0" />      <geometry>
         <box size="0.19 0.28 0.06" />
       </geometry>
@@ -81,4 +92,5 @@
       </geometry>
     </collision>
+<!--
     <collision>
       <origin xyz="-0.062156 -0.002558 0.0125" rpy="0 0 ${radians(32.5)}" />
@@ -92,5 +104,5 @@
         <box size="0.013 0.04 0.025" />
       </geometry>
-    </collision>
+    </collision> -->
   </link>
   <xacro:include filename="$(find mirte_master_description)/urdf/wheel.xacro" />
@@ -193,62 +205,4 @@
     <xacro:include filename="$(find mirte_master_description)/urdf/lidar.xacro" />
   </xacro:if>
-  <xacro:if value="$(arg screen_enable)">
-    <link
-      name="screen">
-      <inertial>
-        <origin
-          xyz="-1.24638847975239E-07 0.0013371323974908 0.00160606068028191"
-          rpy="0 0 0" />
-        <mass
-          value="0.00357270774970056" />
-        <inertia
-          ixx="1.29976980207027E-07"
-          ixy="-1.78182996362165E-11"
-          ixz="-4.24689246841474E-13"
-          iyy="2.09902246549457E-07"
-          iyz="1.92672613573332E-09"
-          izz="3.37075734369407E-07" />
-      </inertial>
-      <visual>
-        <origin
-          xyz="0 0 0"
-          rpy="0 0 0" />
-        <geometry>
-          <mesh
-            filename="package://mirte_master_description/meshes/screen.STL" />
-        </geometry>
-        <material
-          name="">
-          <color
-            rgba="0.768627450980392 0.768627450980392 0.768627450980392 1" />
-        </material>
-      </visual>
-      <collision>
-        <origin
-          xyz="0 0 0"
-          rpy="0 0 0" />
-        <geometry>
-          <mesh
-            filename="package://mirte_master_description/meshes/screen.STL" />
-        </geometry>
-      </collision>
-    </link>
-    <joint
-      name="screen_joint"
-      type="fixed">
-      <origin
-        xyz="0 0.121521156261136 0.0540000000000046"
-        rpy="1.5707963267949 0 -3.14159265358979" />
-      <parent
-        link="frame_link" />
-      <child
-        link="screen" />
-      <axis
-        xyz="0 0 0" />
-    </joint>
-  </xacro:if>
-  <xacro:if value="$(arg flag_enable)">
-    <xacro:include filename="$(find mirte_master_description)/urdf/flag.xacro" />
-  </xacro:if>
   <xacro:if value="$(arg arm_enable)">
     <xacro:include filename="$(find mirte_master_description)/urdf/arm.xacro" />

File: mirte_description/mirte_master_description/urdf/ros2_control.xacro (robot description, xacro)
@@ -87,5 +87,5 @@
     </joint>
     <xacro:if value="$(arg sim)">
-      <joint name="_Gripper_joint_r">
+      <!-- <joint name="_Gripper_joint_r">
         <param name="mimic">gripper_joint</param>
         <param name="multiplier">-1</param>
@@ -107,5 +107,5 @@
         <state_interface name="position" />
         <state_interface name="velocity" />
-      </joint>
+      </joint> -->
     </xacro:if>
 </ros2_control>

Commit message: mmv2 desc: fix tf, wip wheel directions

File: mirte_description/mirte_master_description/urdf/depth_cam.xacro (robot description, xacro)
@@ -30,5 +30,5 @@
       rpy="0 0 2.66843002436935E-05" />
     <parent
-      link="Base" />
+      link="base_link" />
     <child
       link="Depth_camera" />

File: mirte_description/mirte_master_description/urdf/mirte_masterv2.xacro (robot description, xacro)
@@ -3,17 +3,18 @@
      Commit Version: 1.6.0-4-g7f85cfe  Build Version: 1.6.7995.38578
      For more information, please see http://wiki.ros.org/sw_urdf_exporter -->
-<robot xmlns:xacro="http://www.ros.org/wiki/xacro"
+<robot xmlns:xacro="http://www.ros.org/wiki/xacro"  xmlns:gz="http://gazebosim.org/schema"
   name="mirte_master_description">
   <xacro:arg name="front_camera_enable" default="False" />
-  <xacro:arg name="sonar_enable" default="True" />
+  <xacro:arg name="sonar_enable" default="False" />
   <xacro:arg name="lidar_enable" default="True" />
   <xacro:arg name="depth_camera_enable" default="False" />
-  <xacro:arg name="imu_enable" default="True" />
+  <xacro:arg name="imu_enable" default="False" />
   <xacro:arg name="wheels_enable" default="True" />
   <xacro:arg name="sim" default="False" />
-    <xacro:arg name="arm_enable" default="True" />
+    <xacro:arg name="arm_enable" default="False" />
     <xacro:arg name="arm_collisions_enable" default="True" />
     <xacro:arg name="gripper_camera_enable" default="True" />
-  <xacro:include filename="$(find mirte_master_description)/urdf/ros2_control.xacro"/>
+  <xacro:include filename="$(find mirte_master_description)/urdf/mirte_master_base.gazebo.xacro" />
+  <!-- <xacro:include filename="$(find mirte_master_description)/urdf/ros2_control.xacro"/>   -->
   <link
     name="MIRTE_Master">
@@ -107,13 +108,13 @@
       </material>
     </visual> -->
-    <collision>
-      <origin
-        xyz="0 0 0"
-        rpy="0 0 0" />
+    <!-- <collision>
+      <origin
+        xyz="0 0 0"
+        rpy="0 0 0" /> -->
       <!-- <geometry>
         <mesh
           filename="package://mirte_master_description/meshes/Wheels.STL" />
       </geometry> -->
-    </collision>
+    <!-- </collision> -->
   </link>
   <!-- <joint
@@ -439,5 +440,5 @@
   </xacro:if>
   <link
-    name="Base">
+    name="base_link">
     <inertial>
       <origin
@@ -484,8 +485,8 @@
       xyz="0 0 0"
       rpy="0 0 0" />
-    <parent
+    <child
       link="MIRTE_Master" />
-    <child
-      link="Base" />
+    <parent
+      link="base_link" />
     <axis
       xyz="0 0 0" />
@@ -497,5 +498,5 @@
     <xacro:include filename="$(find mirte_master_description)/urdf/ultrasonic.xacro" />
     <joint name="chassis_base_joint" type="fixed">
-      <parent link="Base" />
+      <parent link="base_link" />
       <child link="link_chassis" />
     </joint>
@@ -576,5 +577,5 @@
       rpy="1.5708 0 0" />
     <parent
-      link="Base" />
+      link="base_link" />
     <child
       link="LiDar" />

File: mirte_description/mirte_master_description/urdf/wheel.gazebo.xacro (robot description, xacro)
@@ -1,12 +1,26 @@
 <?xml version="1.0"?>
-<robot xmlns:xacro="http://ros.org/wiki/xacro">
-    <xacro:macro name="wheel_gazebo" params="id">
-        <gazebo reference="wheel_${id}">
+<robot xmlns:xacro="http://ros.org/wiki/xacro"  xmlns:gz="http://gazebosim.org/schema">
+    <xacro:macro name="wheel_gazebo" params="id wheel_type">
+        <gazebo reference="${id}_wheel">
+        <!-- wheel_${id} -->
             <selfCollide>false</selfCollide>
             <gravity>true</gravity>
-            <mu1>0.0</mu1>
+            <mu1>1.0</mu1>
             <mu2>0.0</mu2>
+<xacro:if value="${wheel_type == 'left'}">
             <material>Gazebo/DarkGrey</material>
+                  <fdir1 gz:expressed_in="base_link">1 1 0</fdir1>
+                </xacro:if>
+                <xacro:if value="${wheel_type == 'right'}">
+                            <material>Gazebo/Purple</material>
+                  <fdir1 gz:expressed_in="base_link">-1 1 0</fdir1>
+                </xacro:if>
         </gazebo>
     </xacro:macro>
 </robot>
+<!--
+1 0 0 : beide, dan rondjes
+0 1 0 : beide, ook rondjes
+0 0 1:  beide, originele gebeueren, dan heen en weer
+z doet weinig
+ -->

File: mirte_description/mirte_master_description/urdf/wheel.xacro (robot description, xacro)
@@ -6,4 +6,9 @@
   <link
     name="${name}_wheel">
+    <!-- <inertial>
+          <origin xyz="0 0 ${link_origin}" />
+          <mass value="2">2</mass
+          </inertia>
+        </inertial> -->
     <inertial>
       <origin xyz="0 0 ${link_origin}" />
@@ -33,22 +38,22 @@
       <origin xyz="0 ${link_origin} 0" rpy="${pi/2} 0 0" />
       <geometry>
-        <cylinder radius="${wheel_radius}" length="${wheel_length}" />
+        <sphere radius="${wheel_radius}" />
+        <!-- <cylinder radius="${wheel_radius}" length="${wheel_length}" /> -->
       </geometry>
-      <surface>
+      <!-- <surface>
             <friction>
-              <ode>
-                <mu>1.0</mu>
-                <mu2>0.0</mu2>
+              <!- - <ode> -  ->
+              <!- - sdfa;ladsfkljasfdkjlasfdlkjasfd - ->
+              <mu>1.0</mu>
+                <!- - <mu2>1.0</mu2> - ->
                 <xacro:if value="${wheel_type == 'left'}">
-                  <fdir1 gz:expressed_in="Wheels">-1 -1 0</fdir1>
+                  <fdir1 gz:expressed_in="base_link">1 -1 0</fdir1>
                 </xacro:if>
                 <xacro:if value="${wheel_type == 'right'}">
-                  <fdir1 gz:expressed_in="Wheels">1 1 0</fdir1>
+                  <fdir1 gz:expressed_in="base_link">1 1 0</fdir1>
                 </xacro:if>
-                <!-- <fdir1 gz:expressed_in="Base">1 -1 0</fdir1> -->
-                                <!-- <fdir1 gz:expressed_in="chassis">1 -1 0</fdir1> -->
-              </ode>
+              <!- - </ode> - ->
             </friction>
-          </surface>
+          </surface> -->
     </collision>
   </link>
