Commit message: dunno, mecanum still no workie

File: mirte_description/mirte_master_description/mirte_master.urdf (robot description, URDF)
Before this commit: robot mirte_master, 31 links, 30 joints
Links:
- removed link _Gripper_r
- removed link _gripper_link_l
- removed link _gripper_link_r
- removed link camera_depth_frame
- removed link camera_depth_optical_frame
- removed link camera_link
- removed link camera_rgb_frame
- removed link camera_rgb_optical_frame
- removed link elbow
- removed link frame_link
- removed link front_left_sonar
- removed link front_right_sonar
- removed link gripper
- removed link gripper_camera_link
- removed link gripper_finger_l
- removed link gripper_finger_r
- removed link imu_link
- removed link laser
- removed link lidar_base
- removed link lidar_link
- removed link link_chassis
- removed link rear_left_sonar
- removed link rear_right_sonar
- removed link shoulder_lift
- removed link shoulder_pan
- removed link wrist
- added link LiDar, mass 0.100511981883324
- added link MIRTE_Master, mass 0.087187694310402
- added link Wheels, mass 0.06645993257182
- link base_link: mass None -> 0.045644924765411; geometry visual mesh filename=package://mirte_master_description/meshes/Base.STL
- link front_left_wheel: mass 2.15 -> 0.1; geometry collision sphere radius=0.05; visual mesh filename=package://mirte_master_description/meshes/BR.STL
- link front_right_wheel: mass 2.15 -> 0.1; geometry collision sphere radius=0.05; visual mesh filename=package://mirte_master_description/meshes/BL.STL
- link rear_left_wheel: mass 2.15 -> 0.1; geometry collision sphere radius=0.05; visual mesh filename=package://mirte_master_description/meshes/BL.STL
- link rear_right_wheel: mass 2.15 -> 0.1; geometry collision sphere radius=0.05; visual mesh filename=package://mirte_master_description/meshes/BR.STL
Joints:
- removed joint _Gripper_joint_r
- removed joint _gripper_link_joint_l
- removed joint _gripper_link_joint_r
- removed joint camera_depth_joint
- removed joint camera_depth_optical_joint
- removed joint camera_joint
- removed joint camera_rgb_joint
- removed joint camera_rgb_optical_joint
- removed joint chassis_base_joint
- removed joint elbow_joint
- removed joint frame_base_joint
- removed joint gripper_camera_joint
- removed joint gripper_finger_joint_l
- removed joint gripper_finger_joint_r
- removed joint gripper_joint
- removed joint imu_joint
- removed joint laser_joint
- removed joint lidar_base_joint
- removed joint lidar_joint
- removed joint shoulder_lift_joint
- removed joint shoulder_pan_joint
- removed joint sonar_front_left
- removed joint sonar_front_right
- removed joint sonar_rear_left
- removed joint sonar_rear_right
- removed joint wrist_joint
- added joint Base_joint: type fixed, parent base_link, child MIRTE_Master, origin xyz=0 0 0 rpy=0 0 0, axis 0 0 0
- added joint LiDar_joint: type fixed, parent base_link, child LiDar, origin xyz=0.03167 -0.063182 -0.011397 rpy=1.5708 0 0, axis 0 0 0
- added joint Wheels_joint: type fixed, parent MIRTE_Master, child Wheels, axis 0 0 0
- joint front_left_wheel_joint: axis 0 0 -1 -> 0 1 0; origin xyz=0.153 -0.085 -0.0455 rpy=1.5708 0 -1.5708 -> xyz=0.080503 0.1075 -0.063 rpy=0 0 0; parent frame_link -> Wheels
- joint front_right_wheel_joint: axis 0 0 -1 -> 0 1 0; origin xyz=-0.098 -0.085 -0.0455 rpy=1.5708 0 -1.5708 -> xyz=0.080503 -0.1075 -0.063 rpy=0 0 0; parent frame_link -> Wheels
- joint rear_left_wheel_joint: axis 0 0 -1 -> 0 1 0; origin xyz=0.153 0.085 -0.0455 rpy=1.5708 0 -1.5708 -> xyz=-0.080503 0.1575 -0.063 rpy=0 0 0; parent frame_link -> Wheels
- joint rear_right_wheel_joint: axis 0 0 -1 -> 0 1 0; origin xyz=-0.098 0.085 -0.0455 rpy=1.5708 0 -1.5708 -> xyz=-0.080503 -0.1575 -0.063 rpy=0 0 0; parent frame_link -> Wheels

File: mirte_description/mirte_master_description/urdf/mirte_masterv2.xacro (robot description, xacro)
@@ -60,5 +60,5 @@
   <xacro:property name="wheel_radius" value="0.050" />
   <xacro:property name="wheel_length" value="0.055" />
-  <xacro:property name="wheel_mass" value="2.15" />
+  <xacro:property name="wheel_mass" value="0.15" />
   <xacro:property name="wheel_velocity" value="8" />
   <xacro:property name="wheel_effort" value="5" />
@@ -68,7 +68,7 @@
     name="Wheels_joint"
     type="fixed">
-    <origin
+    <!-- <origin
       xyz="0.0316698713027512 -0.052970257715017 -0.0113974879084128"
-      rpy="1.5707963267949 0 2.66843002434429E-05" />
+      rpy="1.5707963267949 0 2.66843002434429E-05" /> -->
     <parent
       link="MIRTE_Master" />
@@ -200,5 +200,5 @@
       </material>
     </visual>
-    <collision>
+    <!-- <collision>
       <origin
         xyz="0 0 0"
@@ -208,5 +208,5 @@
           filename="package://mirte_master_description/meshes/Wheels.STL" />
       </geometry>
-    </collision>
+    </collision> -->
   </link>
   <joint
@@ -469,5 +469,5 @@
       </material>
     </visual>
-    <collision>
+    <!-- <collision>
       <origin
         xyz="0 0 0"
@@ -477,5 +477,5 @@
           filename="package://mirte_master_description/meshes/Base.STL" />
       </geometry>
-    </collision>
+    </collision> -->
   </link>
   <joint

File: mirte_description/mirte_master_description/urdf/wheel.gazebo.xacro (robot description, xacro)
@@ -1,19 +1,38 @@
 <?xml version="1.0"?>
-<robot xmlns:xacro="http://ros.org/wiki/xacro"  xmlns:gz="http://gazebosim.org/schema">
+<robot xmlns:xacro="http://ros.org/wiki/xacro" xmlns:gz="http://gazebosim.org/schema">
     <xacro:macro name="wheel_gazebo" params="id wheel_type">
         <gazebo reference="${id}_wheel">
-        <!-- wheel_${id} -->
+            <!-- wheel_${id} -->
             <selfCollide>false</selfCollide>
             <gravity>true</gravity>
+            <xacro:if value="${id == 'front_left'}">
+                <!-- -1 x x lijkt ok voor zijwaarts -->
+                                <material>Gazebo/Blue</material><fdir1 gz:expressed_in="MIRTE_Master">1 1 0</fdir1>
             <mu1>1.0</mu1>
             <mu2>0.0</mu2>
-<xacro:if value="${wheel_type == 'left'}">
-            <material>Gazebo/DarkGrey</material>
-                  <fdir1 gz:expressed_in="base_link">1 1 0</fdir1>
-                </xacro:if>
-                <xacro:if value="${wheel_type == 'right'}">
-                            <material>Gazebo/Purple</material>
-                  <fdir1 gz:expressed_in="base_link">-1 1 0</fdir1>
-                </xacro:if>
+            </xacro:if>
+            <xacro:if value="${id == 'front_right'}">
+                                <material>Gazebo/Yellow</material><fdir1 gz:expressed_in="MIRTE_Master">1 -1 0</fdir1>
+            <mu1>1.0</mu1>
+            <mu2>0.0</mu2>
+            </xacro:if>
+            <xacro:if value="${id == 'rear_left'}">
+                                <material>Gazebo/Orange</material><fdir1 gz:expressed_in="MIRTE_Master">1 -1 0</fdir1>
+            <mu1>1.0</mu1>
+            <mu2>0.0</mu2>
+            </xacro:if>
+            <xacro:if value="${id == 'rear_right'}">
+                                <material>Gazebo/Red</material><fdir1 gz:expressed_in="MIRTE_Master">1 1 0</fdir1>
+            <mu1>1.0</mu1>
+            <mu2>0.0</mu2>
+            </xacro:if>
+            <!-- <xacro:if value="${wheel_type == 'left'}">
+                <material>Gazebo/DarkGrey</material>
+                <fdir1 gz:expressed_in="base_link">1 1 0</fdir1>
+            </xacro:if>
+            <xacro:if value="${wheel_type == 'right'}">
+                <material>Gazebo/Purple</material>
+                <fdir1 gz:expressed_in="base_link">-1 1 0</fdir1>
+            </xacro:if> -->
         </gazebo>
     </xacro:macro>

File: mirte_description/mirte_master_description/urdf/wheel.xacro (robot description, xacro)
@@ -12,10 +12,12 @@
         </inertial> -->
     <inertial>
-      <origin xyz="0 0 ${link_origin}" />
-      <mass value="${wheel_mass}" />
+      <!-- <origin xyz="0 0 ${link_origin}" /> -->
+             <origin xyz="0 ${link_origin} 0" rpy="${pi/2} 0 0" />
+<!-- ${wheel_mass * (wheel_radius **2) / 2} -->
+      <mass value="0.1" />
       <inertia
         ixx="${wheel_mass * (3 * (wheel_radius**2) + (wheel_length**2)) / 12}"
         iyy="${wheel_mass * (3 * (wheel_radius**2) + (wheel_length**2)) / 12}"
-        izz="${wheel_mass * (wheel_radius **2) / 2}"
+        izz="${wheel_mass * (3 * (wheel_radius**2) + (wheel_length**2)) / 12}"
         ixy="0" ixz="0" iyz="0" />
     </inertial>
