Commit message: Add lidar & arm gripper parts (need calibration fixes)

File: mirte_description/mirte_master_description/mirte_master.urdf (robot description, URDF)
Before this commit: robot mirte_master_description, 8 links, 7 joints
Links:
- added link Arm, mass 0.438578226451647
- added link Arm_camera, mass 0.00146668134870463
- added link _Gripper_r, mass 0.0127576574866818; collision mesh filename=package://mirte_master_description/meshes/_Gripper_r.STL; visual mesh filename=package://mirte_master_description/meshes/_Gripper_r.STL
- added link _gripper_link_l, mass 0.0025785751096632; collision mesh filename=package://mirte_master_description/meshes/_gripper_link_l.S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; visual mesh filename=package://mirte_master_description/meshes/_gripper_link_l.S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
- added link _gripper_link_r, mass 0.00257857268754656; collision mesh filename=package://mirte_master_description/meshes/_gripper_link_r.S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; visual mesh filename=package://mirte_master_description/meshes/_gripper_link_r.S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
- added link elbow, mass 0.0911215389802598; collision mesh filename=package://mirte_master_description/meshes/Forearm.STL; visual mesh filename=package://mirte_master_description/meshes/Forearm.STL
- added link gripper, mass 0.0109603788959771; collision mesh filename=package://mirte_master_description/meshes/Gripper.STL; visual mesh filename=package://mirte_master_description/meshes/Gripper.STL
- added link gripper_finger_l, mass 0.00531205810762777; collision mesh filename=package://mirte_master_description/meshes/gripper_finger_l.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; visual mesh filename=package://mirte_master_description/meshes/gripper_finger_l.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
- added link gripper_finger_r, mass 0.00531205810762776; collision mesh filename=package://mirte_master_description/meshes/gripper_finger_r.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; visual mesh filename=package://mirte_master_description/meshes/gripper_finger_r.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
- added link shoulder_lift, mass 0.102325054139096; collision mesh filename=package://mirte_master_description/meshes/Upperarm.STL; visual mesh filename=package://mirte_master_description/meshes/Upperarm.STL
- added link shoulder_pan, mass 0.0526781402686753; collision mesh filename=package://mirte_master_description/meshes/z-Rotation.STL; visual mesh filename=package://mirte_master_description/meshes/z-Rotation.STL
- added link wrist, mass 0.0631657082718983; collision mesh filename=package://mirte_master_description/meshes/Wrist.STL; visual mesh filename=package://mirte_master_description/meshes/Wrist.STL
- link MIRTE_Master: mass 0.087187694310402 -> 2.87187694310402
- link Wheels: mass 0.06645993257182 -> 1.06645993257182
- link base_link: mass 0.045644924765411 -> 1.45644924765411
Joints:
- added joint Arm_camera_joint: type fixed, parent wrist, child Arm_camera, origin xyz=0.00808405147922392 -0.0236577575521872 0.0749676192971127 rpy=-7.04933984956096E-05 -0.394897827073442 0.0591050619044624, axis 0 0 1
- added joint Arm_joint: type fixed, parent MIRTE_Master, child Arm, origin xyz=0.00012036 -0.01012 -0.0024812 rpy=1.5708 0 0, axis 0 0 0
- added joint _Gripper_joint_r: type revolute, parent wrist, child _Gripper_r, origin xyz=0.0435 0.012 0.0045 rpy=-1.5708 0 -3.1416, axis 0 -1 0, limit lower=-.25 upper=0.20 effort=2.0 velocity=2.0, mimic joint=gripper_joint multiplier=-1
- added joint _gripper_link_joint_l: type revolute, parent wrist, child _gripper_link_l, origin xyz=0.0605 -0.0205 -0.0055 rpy=1.5708 0 -1.7775, axis 0 -1 0, limit lower=-3.14 upper=3.14 effort=0.0 velocity=0.0, mimic joint=gripper_joint multiplier=-1.4
- added joint _gripper_link_joint_r: type revolute, parent wrist, child _gripper_link_r, origin xyz=0.0605 0.0205 -0.0055 rpy=1.5708 0 -1.3641, axis 0 -1 0, limit lower=-3.14 upper=3.14 effort=0.0 velocity=0.0, mimic joint=gripper_joint multiplier=1.4
- added joint elbow_joint: type revolute, parent shoulder_lift, child elbow, origin xyz=0.036437928080887 0.00180537281653873 0.137006236814825 rpy=0 0 0, axis -0.0590713107275747 0.998253765455679 0, limit lower=-1.5707963267948966 upper=1.5707963267948966 effort=2.0 velocity=2.0
- added joint gripper_finger_joint_l: type fixed, parent _gripper_link_l, child gripper_finger_l, origin xyz=0 0 -0.037 rpy=0 0.20667 0, axis 0 0 1
- added joint gripper_finger_joint_r: type fixed, parent _gripper_link_r, child gripper_finger_r, origin xyz=0 0.01 -0.037 rpy=0 0.20667 3.1416, axis 0 0 1
- added joint gripper_joint: type revolute, parent wrist, child gripper, origin xyz=0.0435 -0.012 0.0045 rpy=-1.5708 0 0, axis 0 -1 0, limit lower=-.20 upper=0.25 effort=2.0 velocity=2.0
- added joint shoulder_lift_joint: type revolute, parent shoulder_pan, child shoulder_lift, origin xyz=0.00380301601043069 0.0313794450114005 0.0332500000000377 rpy=0 -2.66843023091516E-05 0, axis -0.0590713107277822 0.998253765455667 0, limit lower=-1.5707963267948966 upper=1.5707963267948966 effort=2.0 velocity=2.0
- added joint shoulder_pan_joint: type revolute, parent Arm, child shoulder_pan, origin xyz=0.121551322610448 -0.00891627722041789 0.110848128389983 rpy=0 2.66843023091516E-05 0, axis 0 0 1, limit lower=-1.5707963267948966 upper=1.5707963267948966 effort=2.0 velocity=2.0
- added joint wrist_joint: type revolute, parent elbow, child wrist, origin xyz=0.124425999226755 0.000550856546668227 0.0712063710175444 rpy=0 0 0, axis -0.0590713107276118 0.998253765455677 0, limit lower=-1.5707963267948966 upper=1.5707963267948966 effort=2.0 velocity=2.0

File: mirte_description/mirte_master_description/urdf/arm2.xacro (robot description, xacro)
@@ -103,5 +103,5 @@
     <origin
       xyz="0.121551322610448 -0.00891627722041789 0.110848128389983"
-      rpy="0 2.66843023091516E-05 0" />
+      rpy="0 0 0" />
     <parent
       link="Arm" />
@@ -164,5 +164,5 @@
     <origin
       xyz="0.00380301601043069 0.0313794450114005 0.0332500000000377"
-      rpy="0 -2.66843023091516E-05 0" />
+      rpy="0 0 0" />
     <parent
       link="shoulder_pan" />
@@ -300,4 +300,5 @@
         />
   </joint>
+  <xacro:if value="False">
   <link
     name="gripper">
@@ -343,5 +344,5 @@
   </link>
   <joint
-    name="Left_gripper_joint"
+    name="gripper_joint"
     type="revolute">
     <origin
@@ -421,9 +422,349 @@
             velocity="2.0"
         />
-  <!-- <mimic
-      joint="Left_gripper_joint"
-      multiplier="-1"
-      offset="0" /> -->
   </joint>
+  </xacro:if>
+  <link
+        name="gripper">
+        <inertial>
+            <origin
+                xyz="0.0128439388984141 0.00467107677719844 -0.023531822516204"
+                rpy="0 0 0" />
+            <mass
+                value="0.0109603788959771" />
+            <inertia
+                ixx="1.64287457972505E-06"
+                ixy="-2.54915969005551E-10"
+                ixz="-3.17766452649769E-07"
+                iyy="2.96639543247368E-06"
+                iyz="-7.8877045337556E-08"
+                izz="1.49193844890504E-06" />
+        </inertial>
+        <visual>
+            <origin
+                xyz="0 0 0"
+                rpy="0 0 0" />
+            <geometry>
+                <mesh
+                    filename="package://mirte_master_description/meshes/Gripper.STL" />
+            </geometry>
+            <material
+                name="">
+                <color
+                    rgba="0.792156862745098 0.819607843137255 0.933333333333333 1" />
+            </material>
+        </visual>
+        <collision>
+            <origin
+                xyz="0 0 0"
+                rpy="0 0 0" />
+            <geometry>
+                <mesh
+                    filename="package://mirte_master_description/meshes/Gripper.STL" />
+            </geometry>
+        </collision>
+    </link>
+    <joint
+        name="gripper_joint"
+        type="revolute">
+        <origin
+            xyz="0.0435 -0.012 0.0045"
+            rpy="-1.5708 0 0" />
+        <parent
+            link="wrist" />
+        <child
+            link="gripper" />
+        <axis
+            xyz="0 -1 0" />
+        <limit
+            lower="-.20"
+            upper="0.25"
+            effort="2.0"
+            velocity="2.0"
+        />
+    </joint>
+   <link
+        name="_gripper_link_r">
+        <inertial>
+            <origin
+                xyz="-1.28017477174502E-08 0.00327806945611438 -0.015628977594268"
+                rpy="0 0 0" />
+            <mass
+                value="0.00257857268754656" />
+            <inertia
+                ixx="4.78055533789155E-07"
+                ixy="-5.230783542464E-14"
+                ixz="-2.66258471113313E-13"
+                iyy="4.85504704619794E-07"
+                iyz="-3.012555423281E-08"
+                izz="3.42900323604584E-08" />
+        </inertial>
+        <visual>
+            <origin
+                xyz="0 0 0"
+                rpy="0 0 0" />
+            <geometry>
+                <mesh
+                    filename="package://mirte_master_description/meshes/_gripper_link_r.STL" />
+            </geometry>
+            <material
+                name="">
+                <color
+                    rgba="0.792156862745098 0.819607843137255 0.933333333333333 1" />
+            </material>
+        </visual>
+        <collision>
+            <origin
+                xyz="0 0 0"
+                rpy="0 0 0" />
+            <geometry>
+                <mesh
+                    filename="package://mirte_master_description/meshes/_gripper_link_r.STL" />
+            </geometry>
+        </collision>
+    </link>
+    <joint
+        name="_gripper_link_joint_r"
+        type="revolute">
+        <origin
+            xyz="0.0605 0.0205 -0.0055"
+            rpy="1.5708 0 -1.3641" />
+        <parent
+            link="wrist" />
+        <child
+            link="_gripper_link_r" />
+        <axis
+            xyz="0 -1 0" />
+        <limit
+            lower="-3.14"
+            upper="3.14"
+            effort="0.0"
+            velocity="0.0" />
+        <mimic joint="gripper_joint" multiplier="1.4"/>
+    </joint>
+    <link
+        name="gripper_finger_r">
+        <inertial>
+            <origin
+                xyz="0.0053582194655247 0.00456985538673528 -0.0146658643393019"
+                rpy="0 0 0" />
+            <mass
+                value="0.00531205810762776" />
+            <inertia
+                ixx="6.56191216382328E-07"
+                ixy="4.9417968242523E-09"
+                ixz="-1.23756532787867E-07"
+                iyy="7.67327744037516E-07"
+                iyz="3.35637410041389E-08"
+                izz="1.97644006824673E-07" />
+        </inertial>
+        <visual>
+            <origin
+                xyz="0 0 0"
+                rpy="0 0 0" />
+            <geometry>
+                <mesh
+                    filename="package://mirte_master_description/meshes/gripper_finger_r.STL" />
+            </geometry>
+            <material
+                name="">
+                <color
+                    rgba="0.792156862745098 0.819607843137255 0.933333333333333 1" />
+            </material>
+        </visual>
+        <collision>
+            <origin
+                xyz="0 0 0"
+                rpy="0 0 0" />
+            <geometry>
+                <mesh
+                    filename="package://mirte_master_description/meshes/gripper_finger_r.STL" />
+            </geometry>
+        </collision>
+    </link>
+    <joint
+        name="gripper_finger_joint_r"
+        type="fixed">
+        <origin
+            xyz="0 0.01 -0.037"
+            rpy="0 0.20667 3.1416" />
+        <parent
+            link="_gripper_link_r" />
+        <child
+            link="gripper_finger_r" />
+        <axis
+            xyz="0 0 1" />
+    </joint>
+    <link
+        name="_gripper_link_l">
+        <inertial>
+            <origin
+                xyz="-2.05686406795635E-09 0.00327805387383495 -0.0156289677422455"
+                rpy="0 0 0" />
+            <mass
+                value="0.0025785751096632" />
+            <inertia
+                ixx="4.78055731035803E-07"
+                ixy="1.11114248069431E-14"
+                ixz="5.45978048241403E-14"
+                iyy="4.85504889003676E-07"
+                iyz="-3.01256260104972E-08"
+                izz="3.4290092499709E-08" />
+        </inertial>
+        <visual>
+            <origin
+                xyz="0 0 0"
+                rpy="0 0 0" />
+            <geometry>
+                <mesh
+                    filename="package://mirte_master_description/meshes/_gripper_link_l.STL" />
+            </geometry>
+            <material
+                name="">
+                <color
+                    rgba="0.792156862745098 0.819607843137255 0.933333333333333 1" />
+            </material>
+        </visual>
+        <collision>
+            <origin
+                xyz="0 0 0"
+                rpy="0 0 0" />
+            <geometry>
+                <mesh
+                    filename="package://mirte_master_description/meshes/_gripper_link_l.STL" />
+            </geometry>
+        </collision>
+    </link>
+    <joint
+        name="_gripper_link_joint_l"
+        type="revolute">
+        <origin
+            xyz="0.0605 -0.0205 -0.0055"
+            rpy="1.5708 0 -1.7775" />
+        <parent
+            link="wrist" />
+        <child
+            link="_gripper_link_l" />
+        <axis
+            xyz="0 -1 0" />
+        <limit
+            lower="-3.14"
+            upper="3.14"
+            effort="0.0"
+            velocity="0.0" />
+        <mimic joint="gripper_joint" multiplier="-1.4"/>
+    </joint>
+    <link
+        name="gripper_finger_l">
+        <inertial>
+            <origin
+                xyz="0.00535821399237165 0.00543015238565805 -0.0146658496889369"
+                rpy="0 0 0" />
+            <mass
+                value="0.00531205810762777" />
+            <inertia
+                ixx="6.56191216382329E-07"
+                ixy="-4.94179682425222E-09"
+                ixz="-1.23756532787868E-07"
+                iyy="7.67327744037519E-07"
+                iyz="-3.35637410041387E-08"
+                izz="1.97644006824674E-07" />
+        </inertial>
+        <visual>
+            <origin
+                xyz="0 0 0"
+                rpy="0 0 0" />
+            <geometry>
+                <mesh
+                    filename="package://mirte_master_description/meshes/gripper_finger_l.STL" />
+            </geometry>
+            <material
+                name="">
+                <color
+                    rgba="0.792156862745098 0.819607843137255 0.933333333333333 1" />
+            </material>
+        </visual>
+        <collision>
+            <origin
+                xyz="0 0 0"
+                rpy="0 0 0" />
+            <geometry>
+                <mesh
+                    filename="package://mirte_master_description/meshes/gripper_finger_l.STL" />
+            </geometry>
+        </collision>
+    </link>
+    <joint
+        name="gripper_finger_joint_l"
+        type="fixed">
+        <origin
+            xyz="0 0 -0.037"
+            rpy="0 0.20667 0" />
+        <parent
+            link="_gripper_link_l" />
+        <child
+            link="gripper_finger_l" />
+        <axis
+            xyz="0 0 1" />
+    </joint>
+    <link
+        name="_Gripper_r">
+        <inertial>
+            <origin
+                xyz="-0.011058953981311 0.00572378908343621 -0.0203029402870159"
+                rpy="0 0 0" />
+            <mass
+                value="0.0127576574866818" />
+            <inertia
+                ixx="1.91784274511554E-06"
+                ixy="-2.13316668505462E-10"
+                ixz="3.18097729104346E-07"
+                iyy="3.19294602407598E-06"
+                iyz="-1.86219200901589E-07"
+                izz="1.63755141963222E-06" />
+        </inertial>
+        <visual>
+            <origin
+                xyz="0 0 0"
+                rpy="0 0 0" />
+            <geometry>
+                <mesh
+                    filename="package://mirte_master_description/meshes/_Gripper_r.STL" />
+            </geometry>
+            <material
+                name="">
+                <color
+                    rgba="0.792156862745098 0.819607843137255 0.933333333333333 1" />
+            </material>
+        </visual>
+        <collision>
+            <origin
+                xyz="0 0 0"
+                rpy="0 0 0" />
+            <geometry>
+                <mesh
+                    filename="package://mirte_master_description/meshes/_Gripper_r.STL" />
+            </geometry>
+        </collision>
+    </link>
+    <joint
+        name="_Gripper_joint_r"
+        type="revolute">
+        <origin
+            xyz="0.0435 0.012 0.0045"
+            rpy="-1.5708 0 -3.1416" />
+        <parent
+            link="wrist" />
+        <child
+            link="_Gripper_r" />
+        <axis
+            xyz="0 -1 0" />
+        <limit
+            lower="-.25"
+            upper="0.20"
+            effort="2.0"
+            velocity="2.0"
+        />
+        <mimic joint="gripper_joint" multiplier="-1"/>
+    </joint>
   <link
     name="Arm_camera">

File: mirte_description/mirte_master_description/urdf/lidarv2.xacro (robot description, xacro)
@@ -1,4 +1,58 @@
 <?xml version="1.0" encoding="UTF-8"?>
 <robot xmlns:xacro="http://www.ros.org/wiki/xacro">
+  <link
+    name="lidar_base">
+    <inertial>
+      <origin
+        xyz="-3.16279539482045E-07 9.54386088163634E-05 -0.0118651639697618"
+        rpy="0 0 0" />
+      <mass
+        value="0.100511981883324" />
+      <inertia
+        ixx="3.39518064050846E-05"
+        ixy="2.51551620720405E-12"
+        ixz="2.11349409641371E-10"
+        iyy="3.4477810166857E-05"
+        iyz="1.18155796489864E-07"
+        izz="4.19358530903682E-05" />
+    </inertial>
+    <!-- <visual>
+      <origin
+        xyz="0 0 0"
+        rpy="0 0 0" />
+      <geometry>
+        <mesh
+          filename="package://mirte_master_description/meshes/LiDar.STL" />
+      </geometry>
+      <material
+        name="">
+        <color
+          rgba="0.501960784313725 0.501960784313725 0.501960784313725 1" />
+      </material>
+    </visual>
+    <collision>
+      <origin
+        xyz="0 0 0"
+        rpy="0 0 0" />
+      <geometry>
+        <mesh
+          filename="package://mirte_master_description/meshes/LiDar.STL" />
+      </geometry>
+    </collision> -->
+  </link>
+  <joint
+    name="LiDar_joint"
+    type="fixed">
+    <origin
+      xyz="0.03167 -0.063182 -0.011397"
+      rpy="0 0 0" />
+    <parent
+      link="base_link" />
+    <child
+      link="lidar_base" />
+    <axis
+      xyz="0 0 0" />
+  </joint>
+<!--
   <link name="lidar_base">
     <inertial>
@@ -39,6 +93,6 @@
       </geometry>
     </collision>
-  </link>
-  <joint
+  </link> -->
+  <!-- <joint
     name="lidar_base_joint"
     type="fixed">
@@ -51,5 +105,5 @@
       link="lidar_base" />
     <axis xyz="0 0 0" />
-  </joint>
+  </joint> -->
   <link name="lidar_link"></link>
   <joint name="lidar_joint" type="fixed">
@@ -59,4 +113,5 @@
     <axis xyz="0 0 0" />
   </joint>
+  <xacro:if value="$(arg use_correct_laser_frame)">
     <link name="laser"></link>
     <joint name="laser_joint" type="fixed">
@@ -67,8 +122,15 @@
     </joint>
     <xacro:property name="lidar_sensor_link" value="laser" />
+  </xacro:if>
+  <xacro:unless value="$(arg use_correct_laser_frame)">
+    <xacro:property name="lidar_sensor_link" value="lidar_link" />
+  </xacro:unless>
   <gazebo reference="lidar_link">
-        <sensor name="lidar" type="ray">
+        <sensor name="lidar" type="gpu_lidar">
+              <pose relative_to='lidar_link'>0 0 0 0 0 0</pose>
+          <gz_frame_id>lidar_link</gz_frame_id>
+          <topic>/scan</topic>
             <pose> 0 0 0 0 0 0 </pose>
-            <visualize>${visualize_sensors}</visualize>
+            <visualize>true</visualize>
             <update_rate>10</update_rate>
             <ray>
@@ -87,11 +149,4 @@
                 </range>
             </ray>
-            <plugin name="laser_controller" filename="libgazebo_ros_ray_sensor.so">
-                <ros>
-                    <remapping>~/out:=scan</remapping>
-                </ros>
-                <output_type>sensor_msgs/LaserScan</output_type>
-                <frame_name>lidar_link</frame_name>
-            </plugin>
         </sensor>
     </gazebo>

File: mirte_description/mirte_master_description/urdf/mirte_masterv2.xacro (robot description, xacro)
@@ -11,6 +11,7 @@
   <xacro:arg name="imu_enable" default="False" />
   <xacro:arg name="wheels_enable" default="True" />
-  <xacro:arg name="sim" default="False" />
-    <xacro:arg name="arm_enable" default="False" />
+  <xacro:arg name="sim" default="True" />
+  <xacro:arg name="use_correct_laser_frame" default="True" />
+    <xacro:arg name="arm_enable" default="True" />
     <xacro:arg name="arm_collisions_enable" default="True" />
     <xacro:arg name="gripper_camera_enable" default="True" />
@@ -530,56 +531,6 @@
     </xacro:ultrasonic_sensor>
   </xacro:if>
-  <link
-    name="LiDar">
-    <inertial>
-      <origin
-        xyz="-3.16279539482045E-07 9.54386088163634E-05 -0.0118651639697618"
-        rpy="0 0 0" />
-      <mass
-        value="0.100511981883324" />
-      <inertia
-        ixx="3.39518064050846E-05"
-        ixy="2.51551620720405E-12"
-        ixz="2.11349409641371E-10"
-        iyy="3.4477810166857E-05"
-        iyz="1.18155796489864E-07"
-        izz="4.19358530903682E-05" />
-    </inertial>
-    <!-- <visual>
-      <origin
-        xyz="0 0 0"
-        rpy="0 0 0" />
-      <geometry>
-        <mesh
-          filename="package://mirte_master_description/meshes/LiDar.STL" />
-      </geometry>
-      <material
-        name="">
-        <color
-          rgba="0.501960784313725 0.501960784313725 0.501960784313725 1" />
-      </material>
-    </visual>
-    <collision>
-      <origin
-        xyz="0 0 0"
-        rpy="0 0 0" />
-      <geometry>
-        <mesh
-          filename="package://mirte_master_description/meshes/LiDar.STL" />
-      </geometry>
-    </collision> -->
-  </link>
-  <joint
-    name="LiDar_joint"
-    type="fixed">
-    <origin
-      xyz="0.03167 -0.063182 -0.011397"
-      rpy="1.5708 0 0" />
-    <parent
-      link="base_link" />
-    <child
-      link="LiDar" />
-    <axis
-      xyz="0 0 0" />
-  </joint>
+  <xacro:if value="$(arg lidar_enable)">
+    <xacro:include filename="$(find mirte_master_description)/urdf/lidarv2.xacro" />
+  </xacro:if>
 </robot>
