Commit message: Add lidar & arm gripper parts (need calibration fixes)

File: mirte_description/mirte_master_description/urdf/ros2_control.xacro (robot description, xacro)
@@ -13,5 +13,5 @@
 </xacro:macro>
 <xacro:if value="True">
-<ros2_control name="GazeboSimSystem" type="system">
+<ros2_control name="GazeboSimSysteasdfzxcveww3rzdsfem" type="system">
   <!-- <hardware>
     <plugin>gz_ros2_control/GazeboSimSystem</plugin>
@@ -23,5 +23,5 @@
         </xacro:if>
         <xacro:unless value="$(arg sim)">
-          <plugin>mirte_base_control/MirteBaseHWInterface</plugin>
+          <plugin>mirte_base_control/MirteBaseHWInterfasdffsadfxzvcwer34ce</plugin>
           <param name="ticks">$(arg ticks)</param>
         <param name="separate_update_format">${params['separate_update_format']}</param>
@@ -51,5 +51,5 @@
       <hardware>
         <xacro:if value="$(arg sim)">
-          <plugin>gz_ros2_control/GazeboSystem</plugin>
+          <plugin>gz_ros2_control/GazeboSimSystem</plugin>
         </xacro:if>
         <xacro:unless value="$(arg sim)">
@@ -87,5 +87,5 @@
      <hardware>
         <xacro:if value="$(arg sim)">
-          <plugin>gz_ros2_control/GazeboSystem</plugin>
+          <plugin>gz_ros2_control/GazeboSimSystem</plugin>
         </xacro:if>
         <xacro:unless value="$(arg sim)">
@@ -105,6 +105,6 @@
         <state_interface name="position" />
         <state_interface name="velocity" />
-      </joint>
-      <joint name="_gripper_link_joint_l">
+      </joint> -->
+      <!-- <joint name="_gripper_link_joint_l">
         <param name="mimic">gripper_joint</param>
         <param name="multiplier">-1.4</param>
@@ -112,6 +112,6 @@
         <state_interface name="position" />
         <state_interface name="velocity" />
-      </joint>
-      <joint name="_gripper_link_joint_r">
+      </joint> -->
+      <!-- <joint name="_gripper_link_joint_r">
         <param name="mimic">gripper_joint</param>
         <param name="multiplier">1.4</param>
