Commit message: base control config moves

File: mirte_control/mirte_master_base_control/bringup/urdf/base.urdf.xacro (robot description, xacro)
@@ -2,9 +2,9 @@
 <!-- TODO: is this file used/reference somewhere? -->
 <robot xmlns:xacro="http://www.ros.org/wiki/xacro" name="diffdrive_robot">
-    <xacro:property name="yaml_param_file" value="$(find mirte_base_control)/config/control_master.yaml"/>
-    <xacro:property name="params" value="${xacro.load_yaml(yaml_param_file)}"/>
-    <xacro:arg name="ticks" default="${params['ticks']}"/>
+    <!-- Load the YAML parameters, default to current pkg, but when using mirte_bringup, it'll use `mirte_bringup/config/control/...` -->
+    <xacro:arg name="hw_config_file" default="$(find mirte_base_control)/config/control_master.yaml"/>
+    <xacro:property name="params" value="${xacro.load_yaml(hw_config_file)}"/>
 <xacro:macro name="wheel" params="name prefix">
-        <joint name="${prefix}${name}_wheel_joint" type="continuous">
+      <joint name="${prefix}${name}_wheel_joint" type="continuous">
       <parent link="${prefix}base_link"/>
       <child link="${prefix}${name}_wheel"/>
@@ -35,5 +35,5 @@
       <hardware>
         <plugin>mirte_base_control/MirteBaseHWInterface</plugin>
-        <param name="ticks">$(arg ticks)</param>
+        <param name="ticks">$(params['ticks'])</param>
         <param name="separate_update_format">${params['separate_update_format']}</param>
         <!-- Use %s in format strings to replace with joint names -->
